File: ledbadge.sch (KiCad schematic (older format))
At the start: 13 parts

Commit message: Added touch, LEDs, power, and connected CPU to other parts.
Parts:
- added C? (x16): C, symbol C
- added D? (x195): APA102, symbol APA102
- added J? (x4): Conn_01x01, symbol Conn_01x01
- added L?: Ferrite_Bead, symbol Ferrite_Bead
- added R? (x9): R, symbol R
- added SW?: SW_Push, symbol SW_Push
- added U?: MTCH105, symbol MTCH105
Connections:
- net labels added: +3V3, +5V, 5V, ACCEL_INT, LP_MODE_SEL, MOSI_3v3, MOSI_5v_R, SCK100, SCK120, SCK140, SCK160, SCK180, SCK20, SCK200, SCK40, SCK60, SCK80, SCL, SCLK_3v3, SCLK_5V_R, SCO120, SDA, SDO100, SDO120, SDO140, SDO160, SDO180, SDO20, SDO200, SDO40, SDO60, SDO80, SENSITIVITY_ADJ, TOUCH0, TOUCH1, TOUCH2/GUARD, TOUCH2/GUARD_CONTROL, TOUCH3, TOUCH4, VDDA, ~TOUCH0_DET, ~TOUCH1_DET, ~TOUCH3_DET, ~TOUCH4_DET
- wire segments 32 -> 499
Other:
- moved on the sheet: D1, D2, D?, R?, U?

Commit message: Added regulators and battery protection
Parts:
- added C? (x25): C, symbol C
- added C? (x4): CP, symbol CP
- added J? (x2): Conn_01x02, symbol Conn_01x02
- added Q? (x2): Q_NMOS_DGS, symbol Q_NMOS_DGS
- added R? (x9): R, symbol R
- added U?: S-8252_(SOT23), symbol S-8252_(SOT23)
- added U?: L7805, symbol L7805
- added U?: AZ1117-3.3, symbol AZ1117-3.3
Connections:
- net labels added: +BATT, TOUCH2/GC
- wire segments 499 -> 605
Other:
- moved on the sheet: C?, J?, L?, R?, SW?, U?

Commit message: Added SWD header
Parts:
- added J?: Conn_01x06, symbol Conn_01x06
- added R? (x2): R, symbol R
- added R?: 10k, symbol R
Connections:
- net labels added: NRST, SWCLK, SWDIO, SWO, ~TOUCH2/GC
- net labels removed: TOUCH2/GC, TOUCH2/GUARD_CONTROL
- wire segments 605 -> 625
Other:
- moved on the sheet: C?, L?, R?, SW?

Commit message: Added crystal, changed MCU from F417 to F407
Parts:
- removed U?: STM32F417VGTx, LQFP100, symbol STM32F417VGTx
- added C? (x5): C, symbol C
- added C? (x2): 6.8p, symbol C
- added R? (x2): 0, symbol R
- added U?: STM32F407VGTx, LQFP100, symbol STM32F407VGTx
- added Y?: Crystal, symbol Crystal
Connections:
- wire segments 625 -> 655
Other:
- moved on the sheet: C?, L?, R?

Commit message: Added power net labels for level shifter, and added VCC ne
Connections:
- net VCC is gone; now on net +5V: U?.5 (VCC), U?.5 (VCC)
Changed lines of the file:
@@
 	20350 13900 20450 13900
 Wire Wire Line
-	3800 1400 8050 1400
+	3150 1400 8050 1400
 Connection ~ 3800 1400
 Wire Wire Line
@@
 Connection ~ 7800 1400
 Wire Wire Line
-	3800 1000 8050 1000
+	3150 1000 8050 1000
 Connection ~ 3800 1000
 Wire Wire Line
@@
 	16900 10000 17200 10000
 Wire Wire Line
-	17200 8950 17200 10000
+	17200 10000 17200 8950
 Wire Wire Line
 	14750 8950 15450 8950
@@
 	15450 8850 17100 8850
 Wire Wire Line
-	15750 8950 17200 8950
+	17200 8950 15750 8950
 Wire Wire Line
 	14750 9350 17000 9350
@@
 Connection ~ 7600 9200
 Connection ~ 7200 9200
+$Comp
+L VCC #PWR?
+U 1 1 5B1504ED
+P 3500 950
+F 0 "#PWR?" H 3500 800 50  0001 C CNN
+F 1 "VCC" H 3500 1100 50  0000 C CNN
+F 2 "" H 3500 950 50  0001 C CNN
+F 3 "" H 3500 950 50  0001 C CNN
+	1    3500 950
+	1    0    0    -1
+$EndComp
+Wire Wire Line
+	3500 950  3500 1000
+$Comp
+L PWR_FLAG #FLG?
+U 1 1 5B151808
+P 3150 950
+F 0 "#FLG?" H 3150 1025 50  0001 C CNN
+F 1 "PWR_FLAG" H 3150 1100 50  0000 C CNN
+F 2 "" H 3150 950 50  0001 C CNN
+F 3 "" H 3150 950 50  0001 C CNN
+	1    3150 950
+	1    0    0    -1
+$EndComp
+Wire Wire Line
+	3150 950  3150 1000
+Connection ~ 3500 1000
+$Comp
+L PWR_FLAG #FLG?
+U 1 1 5B1534CC
+P 3150 1350
+F 0 "#FLG?" H 3150 1425 50  0001 C CNN
+F 1 "PWR_FLAG" H 3150 1500 50  0000 C CNN
+F 2 "" H 3150 1350 50  0001 C CNN
+F 3 "" H 3150 1350 50  0001 C CNN
+	1    3150 1350
+	1    0    0    -1
+$EndComp
+Wire Wire Line
+	3150 1350 3150 1400
 $EndSCHEMATC

Commit message: Added option for touch sensitivity control from DAC1
Parts:
- added C?: C, symbol C
- added R? (x2): R, symbol R
- added RV?: POT, symbol POT
Connections:
- net +3V3: now also RV?.1
- net GND: now also C?.2, RV?.3
- net SENSITIVITY_ADJ: now also C?.1, R?.2, R?.2
- net DAC_OUT1: now reaches U?.29 (ADC1_IN4/ADC2_IN4/DAC_OUT1/DCMI_HSYNC/I2S3_WS/SPI1_NSS/SPI3_NSS/USART2_CK/USB_OTG_HS_SOF/PA4)
- net DAC_OUT1: now also R?.1
- new net: R?.1, RV?.2

Commit message: Added labels, and fixed a few nets
Parts:
- removed J? (x4): Conn_01x01, symbol Conn_01x01
- added C? (x17): C, symbol C
- added J10, J4, J5, J6, J7, J8, J9: TEST_1P, symbol TEST_1P
- R23: renamed from R?; value R -> 0
- gave numbers to parts that had none: 296
Connections:
- net LP_MODE_SEL is gone; now on net +3V3: U7.4 (MTPM)
- net +5V: now also C?.1, C?.1, C?.1, C?.1, C?.1, C?.1, C?.1, C?.1, C?.1, C?.1, C?.1, C?.1, C?.1, C?.1, C?.1, C?.1, C?.1
- net GND: now also U4.1 (CLKIN), C?.2, C?.2, C?.2, C?.2, C?.2, C?.2, C?.2, C?.2, C?.2, C?.2, C?.2, C?.2, C?.2, C?.2, C?.2, C?.2, C?.2
- net TOUCH2/GUARD: now also J10.1
- net at U4.6 (AUX_SDA): now also J4.1
- net at U4.7 (AUX_SCL): now also J5.1
- net at R24.1: now also J6.1
- net at R25.1: now also J7.1
- net at R26.1: now also J8.1
- net at R27.1: now also J9.1
Other:
- note added: "6DOF IMU"
- note added: "Battery Protection"
- note added: "Populating R23 with a 0ohm resistor\nwill enable the guard funciton\non the MTCH105."
- note added: "Regulators"
- note added: "Sensitivity Control for the touch input"
- note added: "This is actually going to be a SMPS drop-in\nreplacement for the 7805"
- note added: "Touch Detection"
- moved on the sheet: C18, C19, C20, C21, C22, R15, R16

Commit message: Added resistors to most MCU pins for easier bluewire fixing later
Parts:
- added J?: Conn_01x06, symbol Conn_01x06
- added R? (x3): R_Small, symbol R_Small
- added R? (x72): R, symbol R
Connections:
- net +3V3: now also R?.1, R?.1, R?.1; no longer U4.8 (~CS), U7.4 (MTPM)
- net ACCEL_INT: now also R?.1; no longer U6.8 (RCC_OSC32_IN/PC14)
- net DAC_OUT1: now also R?.1; no longer U6.29 (ADC1_IN4/ADC2_IN4/DAC_OUT1/DCMI_HSYNC/I2S3_WS/SPI1_NSS/SPI3_NSS/USART2_CK/USB_OTG_HS_SOF/PA4)
- net GND: now also J?.1 (Pin_1), R?.2
- net MOSI_3v3: now also R?.1; no longer U6.32 (ADC1_IN7/ADC2_IN7/ETH_CRS_DV/ETH_RX_DV/SPI1_MOSI/TIM14_CH1/TIM1_CH1N/TIM3_CH2/TIM8_CH1N/PA7)
- net SCL: now also R?.1; no longer U6.92 (CAN2_TX/DCMI_D5/I2C1_SCL/TIM4_CH1/USART1_TX/PB6)
- net SCLK_3v3: now also R?.2; no longer U6.30 (ADC1_IN5/ADC2_IN5/DAC_OUT2/SPI1_SCK/TIM2_CH1/TIM2_ETR/TIM8_CH1N/USB_OTG_HS_ULPI_CK/PA5)
- net SDA: now also R?.2; no longer U6.93 (DCMI_VSYNC/FSMC_NL/I2C1_SDA/TIM4_CH2/USART1_RX/PB7)
- net SWCLK: now also R?.2; no longer U6.76 (SYS_JTCK-SWCLK/PA14)
- net SWDIO: now also R?.1; no longer U6.72 (SYS_JTMS-SWDIO/PA13)
- net SWO: now also R?.2; no longer U6.89 (I2S3_CK/SPI1_SCK/SPI3_SCK/SYS_JTDO-SWO/TIM2_CH2/PB3)
- net ~TOUCH0_DET: now also R?.2; no longer U6.81 (PD0/CAN1_RX/FSMC_D2/FSMC_DA2)
- net ~TOUCH1_DET: now also R?.1; no longer U6.82 (PD1/CAN1_TX/FSMC_D3/FSMC_DA3)
- net ~TOUCH2/GC: now also R?.2; no longer U6.83 (PD2/DCMI_D11/SDIO_CMD/TIM3_ETR/UART5_RX)
- net ~TOUCH3_DET: now also R?.1; no longer U6.84 (PD3/FSMC_CLK/USART2_CTS)
- net ~TOUCH4_DET: now also R?.1; no longer U6.85 (PD4/FSMC_NOE/USART2_RTS)
- net at U4.9 (AD0/MISO): now also R?.1, R?.2
- net at U6.1 (PE2/ETH_TXD3/FSMC_A23/SYS_TRACECLK): now also R?.1
- net at U6.15 (ADC1_IN10/ADC2_IN10/ADC3_IN10/USB_OTG_HS_ULPI_STP/PC0): now also R?.2
- net at U6.16 (ADC1_IN11/ADC2_IN11/ADC3_IN11/ETH_MDC/PC1): now also R?.1
- net at U6.17 (ADC1_IN12/ADC2_IN12/ADC3_IN12/ETH_TXD2/I2S2_ext_SD/SPI2_MISO/USB_OTG_HS_ULPI_DIR/PC2): now also R?.2
- net at U6.18 (ADC1_IN13/ADC2_IN13/ADC3_IN13/ETH_TX_CLK/I2S2_SD/SPI2_MOSI/USB_OTG_HS_ULPI_NXT/PC3): now also R?.1
- net at U6.2 (PE3/FSMC_A19/SYS_TRACED0): now also R?.2
- net at U6.23 (ADC1_IN0/ADC2_IN0/ADC3_IN0/ETH_CRS/SYS_WKUP/TIM2_CH1/TIM2_ETR/TIM5_CH1/TIM8_ETR/UART4_TX/USART2_CTS/PA0): now also R?.2
- net at U6.24 (ADC1_IN1/ADC2_IN1/ADC3_IN1/ETH_REF_CLK/ETH_RX_CLK/TIM2_CH2/TIM5_CH2/UART4_RX/USART2_RTS/PA1): now also R?.1
- net at U6.25 (ADC1_IN2/ADC2_IN2/ADC3_IN2/ETH_MDIO/TIM2_CH3/TIM5_CH3/TIM9_CH1/USART2_TX/PA2): now also R?.2
- net at U6.26 (ADC1_IN3/ADC2_IN3/ADC3_IN3/ETH_COL/TIM2_CH4/TIM5_CH4/TIM9_CH2/USART2_RX/USB_OTG_HS_ULPI_D0/PA3): now also R?.1
- net at U6.3 (PE4/DCMI_D4/FSMC_A20/SYS_TRACED1): now also R?.1
- net at U6.33 (ADC1_IN14/ADC2_IN14/ETH_RXD0/PC4): now also R?.2
- net at U6.34 (ADC1_IN15/ADC2_IN15/ETH_RXD1/PC5): now also R?.1
- net at U6.38 (PE7/FSMC_D4/FSMC_DA4/TIM1_ETR): now also R?.2
- net at U6.39 (PE8/FSMC_D5/FSMC_DA5/TIM1_CH1N): now also R?.1
- net at U6.4 (PE5/DCMI_D6/FSMC_A21/SYS_TRACED2/TIM9_CH1): now also R?.2
- net at U6.40 (PE9/DAC_EXTI9/FSMC_D6/FSMC_DA6/TIM1_CH1): now also R?.2
- net at U6.41 (PE10/FSMC_D7/FSMC_DA7/TIM1_CH2N): now also R?.1
- net at U6.42 (PE11/ADC1_EXTI11/ADC2_EXTI11/ADC3_EXTI11/FSMC_D8/FSMC_DA8/TIM1_CH2): now also R?.2
- net at U6.43 (PE12/FSMC_D9/FSMC_DA9/TIM1_CH3N): now also R?.1
- net at U6.44 (PE13/FSMC_D10/FSMC_DA10/TIM1_CH3): now also R?.2
- net at U6.45 (PE14/FSMC_D11/FSMC_DA11/TIM1_CH4): now also R?.1
- net at U6.46 (PE15/ADC1_EXTI15/ADC2_EXTI15/ADC3_EXTI15/FSMC_D12/FSMC_DA12/TIM1_BKIN): now also R?.2
- net at U6.47 (ETH_RX_ER/I2C2_SCL/I2S2_CK/SPI2_SCK/TIM2_CH3/USART3_TX/USB_OTG_HS_ULPI_D3/PB10): now also R?.2
- net at U6.48 (ADC1_EXTI11/ADC2_EXTI11/ADC3_EXTI11/ETH_TX_EN/I2C2_SDA/TIM2_CH4/USART3_RX/USB_OTG_HS_ULPI_D4/PB11): now also R?.1
- net at U6.5 (PE6/DCMI_D7/FSMC_A22/SYS_TRACED3/TIM9_CH2): now also R?.1
- net at U6.51 (CAN2_RX/ETH_TXD0/I2C2_SMBA/I2S2_WS/SPI2_NSS/TIM1_BKIN/USART3_CK/USB_OTG_HS_ID/USB_OTG_HS_ULPI_D5/PB12): now also R?.2
- net at U6.52 (CAN2_TX/ETH_TXD1/I2S2_CK/SPI2_SCK/TIM1_CH1N/USART3_CTS/USB_OTG_HS_ULPI_D6/USB_OTG_HS_VBUS/PB13): now also R?.1
- net at U6.53 (I2S2_ext_SD/SPI2_MISO/TIM12_CH1/TIM1_CH2N/TIM8_CH2N/USART3_RTS/USB_OTG_HS_DM/PB14): now also R?.2
- net at U6.54 (ADC1_EXTI15/ADC2_EXTI15/ADC3_EXTI15/I2S2_SD/RTC_REFIN/SPI2_MOSI/TIM12_CH2/TIM1_CH3N/TIM8_CH3N/USB_OTG_HS_DP/PB15): now also R?.1
- net at U6.55 (PD8/FSMC_D13/FSMC_DA13/USART3_TX): now also R?.1
- net at U6.56 (PD9/DAC_EXTI9/FSMC_D14/FSMC_DA14/USART3_RX): now also R?.2
- net at U6.57 (PD10/FSMC_D15/FSMC_DA15/USART3_CK): now also R?.1
- net at U6.58 (PD11/ADC1_EXTI11/ADC2_EXTI11/ADC3_EXTI11/FSMC_A16/FSMC_CLE/USART3_CTS): now also R?.2
- net at U6.59 (PD12/FSMC_A17/FSMC_ALE/TIM4_CH1/USART3_RTS): now also R?.1
- net at U6.60 (PD13/FSMC_A18/TIM4_CH2): now also R?.2
- net at U6.61 (PD14/FSMC_D0/FSMC_DA0/TIM4_CH3): now also R?.1
- net at U6.62 (PD15/ADC1_EXTI15/ADC2_EXTI15/ADC3_EXTI15/FSMC_D1/FSMC_DA1/TIM4_CH4): now also R?.2
- net at U6.63 (DCMI_D0/I2S2_MCK/SDIO_D6/TIM3_CH1/TIM8_CH1/USART6_TX/PC6): now also R?.2
- net at U6.64 (DCMI_D1/I2S3_MCK/SDIO_D7/TIM3_CH2/TIM8_CH2/USART6_RX/PC7): now also R?.1
- net at U6.65 (DCMI_D2/SDIO_D0/TIM3_CH3/TIM8_CH3/USART6_CK/PC8): now also R?.2
- net at U6.66 (DAC_EXTI9/DCMI_D3/I2C3_SDA/I2S_CKIN/RCC_MCO_2/SDIO_D1/TIM3_CH4/TIM8_CH4/PC9): now also R?.1
- net at U6.68 (DAC_EXTI9/DCMI_D0/I2C3_SMBA/TIM1_CH2/USART1_TX/USB_OTG_FS_VBUS/PA9): now also R?.2
- net at U6.69 (DCMI_D1/TIM1_CH3/USART1_RX/USB_OTG_FS_ID/PA10): now also R?.1
- net at U6.7 (ANTI_TAMP/RTC_AF1/PC13): now also R?.1
- net at U6.78 (DCMI_D8/I2S3_CK/SDIO_D2/SPI3_SCK/UART4_TX/USART3_TX/PC10): now also R?.2
- net at U6.79 (ADC1_EXTI11/ADC2_EXTI11/ADC3_EXTI11/DCMI_D4/I2S3_ext_SD/SDIO_D3/SPI3_MISO/UART4_RX/USART3_RX/PC11): now also R?.1
- net at U6.80 (DCMI_D9/I2S3_SD/SDIO_CK/SPI3_MOSI/UART5_TX/USART3_CK/PC12): now also R?.2
- net at U6.86 (PD5/FSMC_NWE/USART2_TX): now also R?.2
- net at U6.87 (PD6/FSMC_NWAIT/USART2_RX): now also R?.1
- net at U6.88 (PD7/FSMC_NCE2/FSMC_NE1/USART2_CK): now also R?.2
- net at U6.95 (CAN1_RX/DCMI_D6/ETH_TXD3/I2C1_SCL/SDIO_D4/TIM10_CH1/TIM4_CH3/PB8): now also R?.2
- net at U6.96 (CAN1_TX/DAC_EXTI9/DCMI_D7/I2C1_SDA/I2S2_WS/SDIO_D5/SPI2_NSS/TIM11_CH1/TIM4_CH4/PB9): now also R?.1
- net at U6.97 (PE0/DCMI_D2/FSMC_NBL0/TIM4_ETR): now also R?.1
- net at U6.98 (PE1/DCMI_D3/FSMC_NBL1): now also R?.2
- new net: R?.2, U4.8 (~CS)
- new net: R?.2, U6.29 (ADC1_IN4/ADC2_IN4/DAC_OUT1/DCMI_HSYNC/I2S3_WS/SPI1_NSS/SPI3_NSS/USART2_CK/USB_OTG_HS_SOF/PA4)
- new net: R?.1, U6.30 (ADC1_IN5/ADC2_IN5/DAC_OUT2/SPI1_SCK/TIM2_CH1/TIM2_ETR/TIM8_CH1N/USB_OTG_HS_ULPI_CK/PA5)
- new net: R?.2, U6.32 (ADC1_IN7/ADC2_IN7/ETH_CRS_DV/ETH_RX_DV/SPI1_MOSI/TIM14_CH1/TIM1_CH1N/TIM3_CH2/TIM8_CH1N/PA7)
- new net: R?.2, U6.72 (SYS_JTMS-SWDIO/PA13)
- new net: R?.1, U6.76 (SYS_JTCK-SWCLK/PA14)
- new net: R?.2, U6.8 (RCC_OSC32_IN/PC14)
- new net: R?.1, U6.81 (PD0/CAN1_RX/FSMC_D2/FSMC_DA2)
- new net: R?.2, U6.82 (PD1/CAN1_TX/FSMC_D3/FSMC_DA3)
- new net: R?.1, U6.83 (PD2/DCMI_D11/SDIO_CMD/TIM3_ETR/UART5_RX)
- new net: R?.2, U6.84 (PD3/FSMC_CLK/USART2_CTS)
- new net: R?.2, U6.85 (PD4/FSMC_NOE/USART2_RTS)
- new net: R?.1, U6.89 (I2S3_CK/SPI1_SCK/SPI3_SCK/SYS_JTDO-SWO/TIM2_CH2/PB3)
- new net: R?.2, U6.92 (CAN2_TX/DCMI_D5/I2C1_SCL/TIM4_CH1/USART1_TX/PB6)
- new net: R?.1, U6.93 (DCMI_VSYNC/FSMC_NL/I2C1_SDA/TIM4_CH2/USART1_RX/PB7)
- new net LP_MODE_SEL: R?.2, U7.4 (MTPM)
- new net SERIAL_CTR: J?.2 (Pin_2)
- new net SERIAL_DTR: J?.6 (Pin_6)
- new net SERIAL_PWR: J?.3 (Pin_3)
- new net SERIAL_RXI: J?.5 (Pin_5), R?.1
- new net SERIAL_TXO: J?.4 (Pin_4), R?.1
- new net USART1_RX: R?.2, R?.2
- new net USART1_TX: R?.1, R?.2
Other:
- note added: "Touch Sensitivity"
- note removed: "Sensitivity Control for the touch input"
- moved on the sheet: C18, C19, C20, C21, C22, C23, C24, C25, C27, C28, C29, C34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
