File: ledbadge.sch (KiCad schematic (older format))
At the start: 426 parts, among them J1 TEST_1P, J10 TEST_1P, J11 TEST_1P, J12 TEST_1P, J13 TEST_1P, J14 TEST_1P, J15 TEST_1P, J16 TEST_1P, J17 TEST_1P, J18 TEST_1P, J19 TEST_1P, J2 TEST_1P, J20 TEST_1P, J21 Conn_01x06, J22 USB_OTG, J23 Conn_01x02, J24 Conn_01x06, J25 Conn_01x02, J28 GS3, J29 TEST_1P, J3 TEST_1P, J30 TEST_1P, J31 TEST_1P, J32 TEST_1P, J33 TEST_1P, J4 TEST_1P, J5 TEST_1P, J6 TEST_1P, J7 TEST_1P, J8 TEST_1P, J9 TEST_1P, Q1 Q_NMOS_GDS, Q2 Q_NMOS_GDS, SW1 SW_Push, U1 74AHCT1G125, U2 74AHCT1G125, U3 S-8252_(SOT23), U4 MPU-6000, U5 L7805, U6 MTCH105, U7 STM32F407VGTx, U8 AZ1117-3.3, X1 Badgelife_shitty_connector, Y1 Crystal

Commit message: changed to 4 layer board, and moved groups on to board outline
Parts:
- C1, C10, C11, C12, C13, C14, C15, C16, C17, C18, C19, C2, C20, C21, C22, C23, C24, C25, C26, C27, C28, C29, C3, C30, C31, C32, C33, C34, C4, C5, C6, C7, C8, C9: footprint Capacitors_SMD:C_0805 -> Capacitors_SMD:C_0603
- J29, J30, J31, J32, J33: footprint Measurement_Points:Measurement_Point_Round-SMD-Pad_Big -> gsg-modules:TESTPOINT-50MIL
Changed lines of the file:
@@
 F 0 "C1" H 3825 1300 50  0000 L CNN
 F 1 "C" H 3825 1100 50  0000 L CNN
-F 2 "Capacitors_SMD:C_0805" H 3838 1050 50  0001 C CNN
+F 2 "Capacitors_SMD:C_0603" H 3838 1050 50  0001 C CNN
 F 3 "" H 3800 1200 50  0001 C CNN
 	1    3800 1200
@@
 F 0 "C2" H 4075 1300 50  0000 L CNN
 F 1 "C" H 4075 1100 50  0000 L CNN
-F 2 "Capacitors_SMD:C_0805" H 4088 1050 50  0001 C CNN
+F 2 "Capacitors_SMD:C_0603" H 4088 1050 50  0001 C CNN
 F 3 "" H 4050 1200 50  0001 C CNN
 	1    4050 1200
@@
 F 0 "C3" H 4325 1300 50  0000 L CNN
 F 1 "C" H 4325 1100 50  0000 L CNN
-F 2 "Capacitors_SMD:C_0805" H 4338 1050 50  0001 C CNN
+F 2 "Capacitors_SMD:C_0603" H 4338 1050 50  0001 C CNN
 F 3 "" H 4300 1200 50  0001 C CNN
 	1    4300 1200
@@
 F 0 "C4" H 4575 1300 50  0000 L CNN
 F 1 "C" H 4575 1100 50  0000 L CNN
-F 2 "Capacitors_SMD:C_0805" H 4588 1050 50  0001 C CNN
+F 2 "Capacitors_SMD:C_0603" H 4588 1050 50  0001 C CNN
 F 3 "" H 4550 1200 50  0001 C CNN
 	1    4550 1200
@@
 F 0 "C5" H 4825 1300 50  0000 L CNN
 F 1 "C" H 4825 1100 50  0000 L CNN
-F 2 "Capacitors_SMD:C_0805" H 4838 1050 50  0001 C CNN
+F 2 "Capacitors_SMD:C_0603" H 4838 1050 50  0001 C CNN
 F 3 "" H 4800 1200 50  0001 C CNN
 	1    4800 1200
@@
 F 0 "C6" H 5075 1300 50  0000 L CNN
 F 1 "C" H 5075 1100 50  0000 L CNN
-F 2 "Capacitors_SMD:C_0805" H 5088 1050 50  0001 C CNN
+F 2 "Capacitors_SMD:C_0603" H 5088 1050 50  0001 C CNN
 F 3 "" H 5050 1200 50  0001 C CNN
 	1    5050 1200
@@
 F 0 "C7" H 5325 1300 50  0000 L CNN
 F 1 "C" H 5325 1100 50  0000 L CNN
-F 2 "Capacitors_SMD:C_0805" H 5338 1050 50  0001 C CNN
+F 2 "Capacitors_SMD:C_0603" H 5338 1050 50  0001 C CNN
 F 3 "" H 5300 1200 50  0001 C CNN
 	1    5300 1200
@@
 F 0 "C8" H 5575 1300 50  0000 L CNN
 F 1 "C" H 5575 1100 50  0000 L CNN
-F 2 "Capacitors_SMD:C_0805" H 5588 1050 50  0001 C CNN
+F 2 "Capacitors_SMD:C_0603" H 5588 1050 50  0001 C CNN
 F 3 "" H 5550 1200 50  0001 C CNN
 	1    5550 1200
@@
 F 0 "C9" H 5825 1300 50  0000 L CNN
 F 1 "C" H 5825 1100 50  0000 L CNN
-F 2 "Capacitors_SMD:C_0805" H 5838 1050 50  0001 C CNN
+F 2 "Capacitors_SMD:C_0603" H 5838 1050 50  0001 C CNN
 F 3 "" H 5800 1200 50  0001 C CNN
 	1    5800 1200
@@
 F 0 "C10" H 6075 1300 50  0000 L CNN
 F 1 "C" H 6075 1100 50  0000 L CNN
-F 2 "Capacitors_SMD:C_0805" H 6088 1050 50  0001 C CNN
+F 2 "Capacitors_SMD:C_0603" H 6088 1050 50  0001 C CNN
 F 3 "" H 6050 1200 50  0001 C CNN
 	1    6050 1200
@@
 F 0 "C11" H 6325 1300 50  0000 L CNN
 F 1 "C" H 6325 1100 50  0000 L CNN
-F 2 "Capacitors_SMD:C_0805" H 6338 1050 50  0001 C CNN
+F 2 "Capacitors_SMD:C_0603" H 6338 1050 50  0001 C CNN
 F 3 "" H 6300 1200 50  0001 C CNN
 	1    6300 1200
@@
 F 0 "C12" H 6575 1300 50  0000 L CNN
 F 1 "C" H 6575 1100 50  0000 L CNN
-F 2 "Capacitors_SMD:C_0805" H 6588 1050 50  0001 C CNN
+F 2 "Capacitors_SMD:C_0603" H 6588 1050 50  0001 C CNN
 F 3 "" H 6550 1200 50  0001 C CNN
 	1    6550 1200
@@
 F 0 "C13" H 6825 1300 50  0000 L CNN
 F 1 "C" H 6825 1100 50  0000 L CNN
-F 2 "Capacitors_SMD:C_0805" H 6838 1050 50  0001 C CNN
+F 2 "Capacitors_SMD:C_0603" H 6838 1050 50  0001 C CNN
 F 3 "" H 6800 1200 50  0001 C CNN
 	1    6800 1200
@@
 F 0 "C14" H 7075 1300 50  0000 L CNN
 F 1 "C" H 7075 1100 50  0000 L CNN
-F 2 "Capacitors_SMD:C_0805" H 7088 1050 50  0001 C CNN
+F 2 "Capacitors_SMD:C_0603" H 7088 1050 50  0001 C CNN
 F 3 "" H 7050 1200 50  0001 C CNN
 	1    7050 1200
@@
 F 0 "C15" H 7325 1300 50  0000 L CNN
 F 1 "C" H 7325 1100 50  0000 L CNN
-F 2 "Capacitors_SMD:C_0805" H 7338 1050 50  0001 C CNN
+F 2 "Capacitors_SMD:C_0603" H 7338 1050 50  0001 C CNN
 F 3 "" H 7300 1200 50  0001 C CNN
 	1    7300 1200
@@
 F 0 "C16" H 7575 1300 50  0000 L CNN
 F 1 "C" H 7575 1100 50  0000 L CNN
-F 2 "Capacitors_SMD:C_0805" H 7588 1050 50  0001 C CNN
+F 2 "Capacitors_SMD:C_0603" H 7588 1050 50  0001 C CNN
 F 3 "" H 7550 1200 50  0001 C CNN
 	1    7550 1200
@@
 F 0 "C17" H 7825 1300 50  0000 L CNN
 F 1 "C" H 7825 1100 50  0000 L CNN
-F 2 "Capacitors_SMD:C_0805" H 7838 1050 50  0001 C CNN
+F 2 "Capacitors_SMD:C_0603" H 7838 1050 50  0001 C CNN
 F 3 "" H 7800 1200 50  0001 C CNN
 	1    7800 1200
@@
 F 0 "J31" H 19200 14170 50  0000 C CNN
 F 1 "TEST_1P" H 19200 14100 50  0000 C CNN
-F 2 "Measurement_Points:Measurement_Point_Round-SMD-Pad_Big" H 19400 13900 50  0001 C CNN
+F 2 "gsg-modules:TESTPOINT-50MIL" H 19400 13900 50  0001 C CNN
 F 3 "" H 19400 13900 50  0001 C CNN
 	1    19200 13900
@@
 F 0 "J29" H 19200 13620 50  0000 C CNN
 F 1 "TEST_1P" H 19200 13550 50  0000 C CNN
-F 2 "Measurement_Points:Measurement_Point_Round-SMD-Pad_Big" H 19400 13350 50  0001 C CNN
+F 2 "gsg-modules:TESTPOINT-50MIL" H 19400 13350 50  0001 C CNN
 F 3 "" H 19400 13350 50  0001 C CNN
 	1    19200 13350
@@
 F 0 "J30" H 20450 13620 50  0000 C CNN
 F 1 "TEST_1P" H 20450 13550 50  0000 C CNN
-F 2 "Measurement_Points:Measurement_Point_Round-SMD-Pad_Big" H 20650 13350 50  0001 C CNN
+F 2 "gsg-modules:TESTPOINT-50MIL" H 20650 13350 50  0001 C CNN
 F 3 "" H 20650 13350 50  0001 C CNN
 	1    20450 13350
@@
 F 0 "J32" H 20450 14170 50  0000 C CNN
 F 1 "TEST_1P" H 20450 14100 50  0000 C CNN
-F 2 "Measurement_Points:Measurement_Point_Round-SMD-Pad_Big" H 20650 13900 50  0001 C CNN
+F 2 "gsg-modules:TESTPOINT-50MIL" H 20650 13900 50  0001 C CNN
 F 3 "" H 20650 13900 50  0001 C CNN
 	1    20450 13900
@@
 F 0 "J33" H 19900 14770 50  0000 C CNN
 F 1 "TEST_1P" H 19900 14700 50  0000 C CNN
-F 2 "Measurement_Points:Measurement_Point_Round-SMD-Pad_Big" H 20100 14500 50  0001 C CNN
+F 2 "gsg-modules:TESTPOINT-50MIL" H 20100 14500 50  0001 C CNN
 F 3 "" H 20100 14500 50  0001 C CNN
 	1    19900 14500
@@
 F 0 "C18" H 9175 1300 50  0000 L CNN
 F 1 "C" H 9175 1100 50  0000 L CNN
-F 2 "Capacitors_SMD:C_0805" H 9188 1050 50  0001 C CNN
+F 2 "Capacitors_SMD:C_0603" H 9188 1050 50  0001 C CNN
 F 3 "" H 9150 1200 50  0001 C CNN
 	1    9150 1200
@@
 F 0 "C19" H 9425 1300 50  0000 L CNN
 F 1 "C" H 9425 1100 50  0000 L CNN
-F 2 "Capacitors_SMD:C_0805" H 9438 1050 50  0001 C CNN
+F 2 "Capacitors_SMD:C_0603" H 9438 1050 50  0001 C CNN
 F 3 "" H 9400 1200 50  0001 C CNN
 	1    9400 1200
@@
 F 0 "C20" H 9675 1300 50  0000 L CNN
 F 1 "C" H 9675 1100 50  0000 L CNN
-F 2 "Capacitors_SMD:C_0805" H 9688 1050 50  0001 C CNN
+F 2 "Capacitors_SMD:C_0603" H 9688 1050 50  0001 C CNN
 F 3 "" H 9650 1200 50  0001 C CNN
 	1    9650 1200
@@
 F 0 "C21" H 9925 1300 50  0000 L CNN
 F 1 "C" H 9925 1100 50  0000 L CNN
-F 2 "Capacitors_SMD:C_0805" H 9938 1050 50  0001 C CNN
+F 2 "Capacitors_SMD:C_0603" H 9938 1050 50  0001 C CNN
 F 3 "" H 9900 1200 50  0001 C CNN
 	1    9900 1200
@@
 F 0 "C22" H 10175 1300 50  0000 L CNN
 F 1 "C" H 10175 1100 50  0000 L CNN
-F 2 "Capacitors_SMD:C_0805" H 10188 1050 50  0001 C CNN
+F 2 "Capacitors_SMD:C_0603" H 10188 1050 50  0001 C CNN
 F 3 "" H 10150 1200 50  0001 C CNN
 	1    10150 1200
@@
 F 0 "C23" H 10425 1300 50  0000 L CNN
 F 1 "C" H 10425 1100 50  0000 L CNN
-F 2 "Capacitors_SMD:C_0805" H 10438 1050 50  0001 C CNN
+F 2 "Capacitors_SMD:C_0603" H 10438 1050 50  0001 C CNN
 F 3 "" H 10400 1200 50  0001 C CNN
 	1    10400 1200
@@
 F 0 "C24" H 10675 1300 50  0000 L CNN
 F 1 "C" H 10675 1100 50  0000 L CNN
-F 2 "Capacitors_SMD:C_0805" H 10688 1050 50  0001 C CNN
+F 2 "Capacitors_SMD:C_0603" H 10688 1050 50  0001 C CNN
 F 3 "" H 10650 1200 50  0001 C CNN
 	1    10650 1200
@@
 F 0 "C25" H 10925 1300 50  0000 L CNN
 F 1 "C" H 10925 1100 50  0000 L CNN
-F 2 "Capacitors_SMD:C_0805" H 10938 1050 50  0001 C CNN
+F 2 "Capacitors_SMD:C_0603" H 10938 1050 50  0001 C CNN
 F 3 "" H 10900 1200 50  0001 C CNN
 	1    10900 1200
@@
 F 0 "C26" H 11175 1300 50  0000 L CNN
 F 1 "C" H 11175 1100 50  0000 L CNN
-F 2 "Capacitors_SMD:C_0805" H 11188 1050 50  0001 C CNN
+F 2 "Capacitors_SMD:C_0603" H 11188 1050 50  0001 C CNN
 F 3 "" H 11150 1200 50  0001 C CNN
 	1    11150 1200
@@
 F 0 "C27" H 11425 1300 50  0000 L CNN
 F 1 "C" H 11425 1100 50  0000 L CNN
-F 2 "Capacitors_SMD:C_0805" H 11438 1050 50  0001 C CNN
+F 2 "Capacitors_SMD:C_0603" H 11438 1050 50  0001 C CNN
 F 3 "" H 11400 1200 50  0001 C CNN
 	1    11400 1200
@@
 F 0 "C28" H 11675 1300 50  0000 L CNN
 F 1 "C" H 11675 1100 50  0000 L CNN
-F 2 "Capacitors_SMD:C_0805" H 11688 1050 50  0001 C CNN
+F 2 "Capacitors_SMD:C_0603" H 11688 1050 50  0001 C CNN
 F 3 "" H 11650 1200 50  0001 C CNN
 	1    11650 1200
@@
 F 0 "C29" H 11925 1300 50  0000 L CNN
 F 1 "C" H 11925 1100 50  0000 L CNN
-F 2 "Capacitors_SMD:C_0805" H 11938 1050 50  0001 C CNN
+F 2 "Capacitors_SMD:C_0603" H 11938 1050 50  0001 C CNN
 F 3 "" H 11900 1200 50  0001 C CNN
 	1    11900 1200
@@
 F 0 "C30" H 12175 1300 50  0000 L CNN
 F 1 "C" H 12175 1100 50  0000 L CNN
-F 2 "Capacitors_SMD:C_0805" H 12188 1050 50  0001 C CNN
+F 2 "Capacitors_SMD:C_0603" H 12188 1050 50  0001 C CNN
 F 3 "" H 12150 1200 50  0001 C CNN
 	1    12150 1200
@@
 F 0 "C31" H 12425 1300 50  0000 L CNN
 F 1 "C" H 12425 1100 50  0000 L CNN
-F 2 "Capacitors_SMD:C_0805" H 12438 1050 50  0001 C CNN
+F 2 "Capacitors_SMD:C_0603" H 12438 1050 50  0001 C CNN
 F 3 "" H 12400 1200 50  0001 C CNN
 	1    12400 1200
@@
 F 0 "C32" H 12675 1300 50  0000 L CNN
 F 1 "C" H 12675 1100 50  0000 L CNN
-F 2 "Capacitors_SMD:C_0805" H 12688 1050 50  0001 C CNN
+F 2 "Capacitors_SMD:C_0603" H 12688 1050 50  0001 C CNN
 F 3 "" H 12650 1200 50  0001 C CNN
 	1    12650 1200
@@
 F 0 "C33" H 12925 1300 50  0000 L CNN
 F 1 "C" H 12925 1100 50  0000 L CNN
-F 2 "Capacitors_SMD:C_0805" H 12938 1050 50  0001 C CNN
+F 2 "Capacitors_SMD:C_0603" H 12938 1050 50  0001 C CNN
 F 3 "" H 12900 1200 50  0001 C CNN
 	1    12900 1200
@@
 F 0 "C34" H 13175 1300 50  0000 L CNN
 F 1 "C" H 13175 1100 50  0000 L CNN
-F 2 "Capacitors_SMD:C_0805" H 13188 1050 50  0001 C CNN
+F 2 "Capacitors_SMD:C_0603" H 13188 1050 50  0001 C CNN
 F 3 "" H 13150 1200 50  0001 C CNN
 	1    13150 1200
