File: ledbadge.sch (KiCad schematic (older format))
At the start: 426 parts, among them J1 TEST_1P, J10 TEST_1P, J11 TEST_1P, J12 TEST_1P, J13 TEST_1P, J14 TEST_1P, J15 TEST_1P, J16 TEST_1P, J17 TEST_1P, J18 TEST_1P, J19 TEST_1P, J2 TEST_1P, J20 TEST_1P, J21 Conn_01x06, J22 USB_OTG, J23 Conn_01x02, J24 Conn_01x06, J25 Conn_01x02, J28 GS3, J29 TEST_1P, J3 TEST_1P, J30 TEST_1P, J31 TEST_1P, J32 TEST_1P, J33 TEST_1P, J4 TEST_1P, J5 TEST_1P, J6 TEST_1P, J7 TEST_1P, J8 TEST_1P, J9 TEST_1P, Q1 Q_NMOS_GDS, Q2 Q_NMOS_GDS, SW1 SW_Push, U1 74AHCT1G125, U2 74AHCT1G125, U3 S-8252_(SOT23), U4 MPU-6000, U5 L7805, U6 MTCH105, U7 STM32F407VGTx, U8 AZ1117-3.3, X1 Badgelife_shitty_connector, Y1 Crystal

Commit message: More part placement, more routing, new board outline
Parts:
- J21, J24: footprint Pin_Headers:Pin_Header_Angled_1x06_Pitch1.27mm -> Pin_Headers:Pin_Header_Straight_1x06_Pitch2.54mm_SMD_Pin1Left
Changed lines of the file:
@@
 F 0 "J21" H 13650 8500 50  0000 C CNN
 F 1 "Conn_01x06" H 13650 7800 50  0000 C CNN
-F 2 "Pin_Headers:Pin_Header_Angled_1x06_Pitch1.27mm" H 13650 8200 50  0001 C CNN
+F 2 "Pin_Headers:Pin_Header_Straight_1x06_Pitch2.54mm_SMD_Pin1Left" H 13650 8200 50  0001 C CNN
 F 3 "" H 13650 8200 50  0001 C CNN
 	1    13650 8200
@@
 F 0 "J24" H 13650 9400 50  0000 C CNN
 F 1 "Conn_01x06" H 13650 8700 50  0000 C CNN
-F 2 "Pin_Headers:Pin_Header_Angled_1x06_Pitch1.27mm" H 13650 9100 50  0001 C CNN
+F 2 "Pin_Headers:Pin_Header_Straight_1x06_Pitch2.54mm_SMD_Pin1Left" H 13650 9100 50  0001 C CNN
 F 3 "" H 13650 9100 50  0001 C CNN
 	1    13650 9100

Commit message: Fixing DRC and unconnected nets
Connections:
- net +5V: now also C64.1, C65.1, C66.1, J28.2 (G2), U8.3 (VI); no longer C61.1, C62.1, C63.1, J28.1 (G1), U5.3 (OUT)
- new net: C61.1, C62.1, C63.1, J28.1 (G1), U5.3 (OUT)
Changed lines of the file:
@@
 L +5V #PWR050
 U 1 1 5B140BD5
-P 16450 11550
-F 0 "#PWR050" H 16450 11400 50  0001 C CNN
-F 1 "+5V" H 16450 11690 50  0000 C CNN
-F 2 "" H 16450 11550 50  0001 C CNN
-F 3 "" H 16450 11550 50  0001 C CNN
-	1    16450 11550
+P 15400 12850
+F 0 "#PWR050" H 15400 12700 50  0001 C CNN
+F 1 "+5V" H 15400 12990 50  0000 C CNN
+F 2 "" H 15400 12850 50  0001 C CNN
+F 3 "" H 15400 12850 50  0001 C CNN
+	1    15400 12850
 	1    0    0    -1
 $EndComp
@@
 Text Label 11600 8850 2    60   ~ 0
 SDA2
-$Comp
-L +5V #PWR069
-U 1 1 5B168232
-P 14700 12750
-F 0 "#PWR069" H 14700 12600 50  0001 C CNN
-F 1 "+5V" H 14700 12890 50  0000 C CNN
-F 2 "" H 14700 12750 50  0001 C CNN
-F 3 "" H 14700 12750 50  0001 C CNN
-	1    14700 12750
-	1    0    0    -1
-$EndComp
 NoConn ~ 12000 10900
 NoConn ~ 12000 11100
@@
 	15100 13100 15800 13100
 Wire Wire Line
-	15400 13250 15400 13100
+	15400 12850 15400 13250
 Connection ~ 15400 13100
 Wire Wire Line
@@
 Connection ~ 14600 11650
 Wire Wire Line
-	15650 11650 16450 11650
+	15650 11650 16800 11650
 Wire Wire Line
 	15850 11650 15850 11800
@@
 	16150 11650 16150 11800
 Connection ~ 15850 11650
-Wire Wire Line
-	16450 11550 16450 11800
 Connection ~ 16150 11650
 Wire Wire Line
@@
 Connection ~ 15100 13100
 Connection ~ 17150 13100
-Connection ~ 16450 11650
 Wire Wire Line
 	13250 12100 13450 12100
@@
 	3950 8350 4500 8350
 Wire Wire Line
-	14750 12850 14700 12850
-Wire Wire Line
-	14700 12850 14700 12750
-Wire Wire Line
 	14750 13050 14650 13050
 Wire Wire Line
@@
 Wire Wire Line
 	9000 8650 9050 8650
+Wire Wire Line
+	16450 11650 16450 11800
+Wire Wire Line
+	14750 12850 14650 12850
+Wire Wire Line
+	14650 12850 14650 12450
+Wire Wire Line
+	14650 12450 16800 12450
+Wire Wire Line
+	16800 12450 16800 11650
+Connection ~ 16450 11650
 $EndSCHEMATC
