File: ledbadge.kicad_pcb (KiCad board)
At the start: 2 copper layers, 0 parts

Commit message: Fixed one 6pin header footprint
Parts:
- added C1: C, Capacitors_SMD:C_0805, F.Cu at (212.7, 114.9)
- added C10: C, Capacitors_SMD:C_0805, F.Cu at (225.0, 98.7)
- added C11: C, Capacitors_SMD:C_0805, F.Cu at (160.8, 152.3)
- added C12: C, Capacitors_SMD:C_0805, F.Cu at (196.9, 115.2)
- added C13: C, Capacitors_SMD:C_0805, F.Cu at (213.2, 98.8)
- added C14: C, Capacitors_SMD:C_0805, F.Cu at (168.9, 143.3)
- added C15: C, Capacitors_SMD:C_0805, F.Cu at (182.4, 130.1)
- added C16: C, Capacitors_SMD:C_0805, F.Cu at (217.8, 93.4)
- added C17: C, Capacitors_SMD:C_0805, F.Cu at (228.5, 82.5)
- added C18: C, Capacitors_SMD:C_0805, F.Cu at (176.4, 135.0)
- added C19: C, Capacitors_SMD:C_0805, F.Cu at (186.0, 124.6)
- added C2: C, Capacitors_SMD:C_0805, F.Cu at (196.2, 131.1)
- added C20: C, Capacitors_SMD:C_0805, F.Cu at (156.8, 152.3)
- added C21: C, Capacitors_SMD:C_0805, F.Cu at (205.4, 104.3)
- added C22: C, Capacitors_SMD:C_0805, F.Cu at (222.1, 87.9)
- added C23: C, Capacitors_SMD:C_0805, F.Cu at (200.4, 109.7)
- added C24: C, Capacitors_SMD:C_0805, F.Cu at (172.5, 135.0)
- added C25: C, Capacitors_SMD:C_0805, F.Cu at (209.3, 104.3)
- added C26: C, Capacitors_SMD:C_0805, F.Cu at (164.7, 148.8)
- added C27: C, Capacitors_SMD:C_0805, F.Cu at (188.3, 135.2)
- added C28: C, Capacitors_SMD:C_0805, F.Cu at (172.6, 150.9)
- added C29: C, Capacitors_SMD:C_0805, F.Cu at (176.8, 146.0)
- added C3: C, Capacitors_SMD:C_0805, F.Cu at (184.7, 140.7)
- added C30: C, Capacitors_SMD:C_0805, F.Cu at (197.8, 125.8)
- added C31: C, Capacitors_SMD:C_0805, F.Cu at (201.8, 120.3)
- added C32: C, Capacitors_SMD:C_0805, F.Cu at (212.3, 109.6)
- added C33: C, Capacitors_SMD:C_0805, F.Cu at (168.7, 154.1)
- added C34: C, Capacitors_SMD:C_0805, F.Cu at (217.2, 104.1)
- added C35: C, Capacitors_SMD:C_0805, F.Cu at (180.8, 140.7)
- added C36: C, Capacitors_SMD:C_0805, F.Cu at (176.8, 140.7)
- added C37: C, Capacitors_SMD:C_0805, F.Cu at (204.8, 115.0)
- added C38: C, Capacitors_SMD:C_0805, F.Cu at (184.3, 135.4)
- added C39: C, Capacitors_SMD:C_0805, F.Cu at (193.9, 125.8)
- added C4: C, Capacitors_SMD:C_0805, F.Cu at (221.2, 104.0)
- added C40: C, Capacitors_SMD:C_0805, F.Cu at (221.1, 98.7)
- added C41: C, Capacitors_SMD:C_0805, F.Cu at (225.7, 93.2)
- added C42: C, Capacitors_SMD:C_0805, F.Cu at (164.7, 154.1)
- added C43: C, Capacitors_SMD:C_0805, F.Cu at (172.9, 145.6)
- added C44: C, Capacitors_SMD:C_0805, F.Cu at (208.3, 109.6)
- added C45: C, Capacitors_SMD:C_0805, F.Cu at (184.7, 146.0)
- added C46: C, Capacitors_SMD:C_0805, F.Cu at (200.1, 131.1)
- added C47: C, Capacitors_SMD:C_0805, F.Cu at (216.6, 114.7)
- added C48: C, Capacitors_SMD:C_0805, F.Cu at (205.7, 125.6)
- added C49: C, Capacitors_SMD:C_0805, F.Cu at (180.5, 151.3)
- added C5: C, Capacitors_SMD:C_0805, F.Cu at (216.2, 109.4)
- added C50: C, Capacitors_SMD:C_0805, F.Cu at (176.6, 151.3)
- added C51: C, Capacitors_SMD:C_0805, F.Cu at (172.6, 156.2)
- added C52: C, Capacitors_SMD:C_0805, F.Cu at (192.2, 136.4)
- added C53: C, Capacitors_SMD:C_0805, F.Cu at (201.8, 125.6)
- added C54: C, Capacitors_SMD:C_0805, F.Cu at (226.0, 87.9)
- added C55: 6.8p, Capacitors_SMD:C_0805, F.Cu at (204.4, 109.7)
- added C56: C, Capacitors_SMD:C_0805, F.Cu at (221.8, 93.4)
- added C57: 6.8p, Capacitors_SMD:C_0805, F.Cu at (189.9, 124.6)
- added C58: CP, Capacitors_Tantalum_SMD:CP_Tantalum_Case-E_EIA-7260-38_Reflow, F.Cu at (45.7, 172.7)
- added C59: C, Capacitors_SMD:C_0805, F.Cu at (172.9, 140.3)
- added C6: C, Capacitors_SMD:C_0805, F.Cu at (205.7, 120.3)
- added C60: C, Capacitors_SMD:C_0805, F.Cu at (200.8, 115.0)
- added C61: CP, Capacitors_Tantalum_SMD:CP_Tantalum_Case-E_EIA-7260-38_Reflow, F.Cu at (164.0, 93.6)
- added C62: C, Capacitors_SMD:C_0805, F.Cu at (217.1, 98.8)
- added C63: C, Capacitors_SMD:C_0805, F.Cu at (186.4, 129.9)
- added C64: CP, Capacitors_Tantalum_SMD:CP_Tantalum_Case-B_EIA-3528-21_Reflow, F.Cu at (114.3, 154.8)
- added C65: C, Capacitors_SMD:C_0805, F.Cu at (180.4, 135.4)
- added C66: C, Capacitors_SMD:C_0805, F.Cu at (168.7, 148.8)
- added C67: CP, Capacitors_Tantalum_SMD:CP_Tantalum_Case-B_EIA-3528-21_Reflow, F.Cu at (168.7, 103.9)
- added C68: C, Capacitors_SMD:C_0805, F.Cu at (213.3, 104.1)
- added C69: C, Capacitors_SMD:C_0805, F.Cu at (193.9, 120.5)
- added C7: C, Capacitors_SMD:C_0805, F.Cu at (180.8, 146.0)
- added C70: C, Capacitors_SMD:C_0805, F.Cu at (197.8, 120.5)
- added C8: C, Capacitors_SMD:C_0805, F.Cu at (192.2, 131.1)
- added C9: C, Capacitors_SMD:C_0805, F.Cu at (208.7, 114.9)
- added D1: APA102, gsg-modules:APA102-2020, F.Cu at (222.5, 154.1)
- added D10: APA102, gsg-modules:APA102-2020, F.Cu at (220.0, 146.0)
- added D100: APA102, gsg-modules:APA102-2020, F.Cu at (195.6, 148.8)
- added D101: APA102, gsg-modules:APA102-2020, F.Cu at (226.5, 117.0)
- added D102: APA102, gsg-modules:APA102-2020, F.Cu at (223.6, 121.7)
- added D103: APA102, gsg-modules:APA102-2020, F.Cu at (220.7, 124.4)
- added D104: APA102, gsg-modules:APA102-2020, F.Cu at (206.4, 129.8)
- added D105: APA102, gsg-modules:APA102-2020, F.Cu at (220.0, 116.3)
- added D106: APA102, gsg-modules:APA102-2020, F.Cu at (222.9, 113.6)
- added D107: APA102, gsg-modules:APA102-2020, F.Cu at (220.0, 113.6)
- added D108: APA102, gsg-modules:APA102-2020, F.Cu at (203.5, 129.8)
- added D109: APA102, gsg-modules:APA102-2020, F.Cu at (184.0, 150.2)
- added D11: APA102, gsg-modules:APA102-2020, F.Cu at (210.9, 154.2)
- added D110: APA102, gsg-modules:APA102-2020, F.Cu at (210.9, 156.9)
- added D111: APA102, gsg-modules:APA102-2020, F.Cu at (218.8, 148.8)
- added D112: APA102, gsg-modules:APA102-2020, F.Cu at (228.7, 138.6)
- added D113: APA102, gsg-modules:APA102-2020, F.Cu at (215.9, 151.5)
- added D114: APA102, gsg-modules:APA102-2020, F.Cu at (225.8, 141.3)
- added D115: APA102, gsg-modules:APA102-2020, F.Cu at (222.9, 143.3)
- added D116: APA102, gsg-modules:APA102-2020, F.Cu at (196.8, 138.0)
- added D117: APA102, gsg-modules:APA102-2020, F.Cu at (201.4, 135.3)
- added D118: APA102, gsg-modules:APA102-2020, F.Cu at (184.0, 152.9)
- added D119: APA102, gsg-modules:APA102-2020, F.Cu at (186.9, 150.2)
- added D12: APA102, gsg-modules:APA102-2020, F.Cu at (208.0, 156.9)
- added D120: APA102, gsg-modules:APA102-2020, F.Cu at (203.5, 132.5)
- added D121: APA102, gsg-modules:APA102-2020, F.Cu at (228.7, 114.3)
- added D122: APA102, gsg-modules:APA102-2020, F.Cu at (196.8, 146.1)
- added D123: APA102, gsg-modules:APA102-2020, F.Cu at (223.6, 119.0)
- added D124: APA102, gsg-modules:APA102-2020, F.Cu at (220.7, 121.7)
- added D125: APA102, gsg-modules:APA102-2020, F.Cu at (217.8, 124.4)
- added D126: APA102, gsg-modules:APA102-2020, F.Cu at (215.1, 127.2)
- added D127: APA102, gsg-modules:APA102-2020, F.Cu at (212.2, 129.9)
- added D128: APA102, gsg-modules:APA102-2020, F.Cu at (202.6, 138.0)
- added D129: APA102, gsg-modules:APA102-2020, F.Cu at (196.8, 143.4)
- added D13: APA102, gsg-modules:APA102-2020, F.Cu at (228.7, 135.9)
- added D130: APA102, gsg-modules:APA102-2020, F.Cu at (192.7, 148.7)
- added D131: APA102, gsg-modules:APA102-2020, F.Cu at (184.8, 155.6)
- added D132: APA102, gsg-modules:APA102-2020, F.Cu at (193.9, 146.0)
- added D133: APA102, gsg-modules:APA102-2020, F.Cu at (181.9, 155.6)
- added D134: APA102, gsg-modules:APA102-2020, F.Cu at (204.3, 135.2)
- added D135: APA102, gsg-modules:APA102-2020, F.Cu at (220.7, 119.0)
- added D136: APA102, gsg-modules:APA102-2020, F.Cu at (217.8, 121.7)
- added D137: APA102, gsg-modules:APA102-2020, F.Cu at (189.8, 148.7)
- added D138: APA102, gsg-modules:APA102-2020, F.Cu at (186.9, 152.9)
- added D139: APA102, gsg-modules:APA102-2020, F.Cu at (214.9, 124.5)
- added D14: APA102, gsg-modules:APA102-2020, F.Cu at (215.9, 148.8)
- added D140: APA102, gsg-modules:APA102-2020, F.Cu at (209.3, 129.9)
- added D141: APA102, gsg-modules:APA102-2020, F.Cu at (218.0, 129.8)
- added D142: APA102, gsg-modules:APA102-2020, F.Cu at (215.1, 132.6)
- added D143: APA102, gsg-modules:APA102-2020, F.Cu at (208.4, 140.7)
- added D144: APA102, gsg-modules:APA102-2020, F.Cu at (226.5, 122.4)
- added D145: APA102, gsg-modules:APA102-2020, F.Cu at (205.5, 143.3)
- added D146: APA102, gsg-modules:APA102-2020, F.Cu at (202.6, 146.1)
- added D147: APA102, gsg-modules:APA102-2020, F.Cu at (223.6, 124.4)
- added D148: APA102, gsg-modules:APA102-2020, F.Cu at (220.9, 127.1)
- added D149: APA102, gsg-modules:APA102-2020, F.Cu at (226.7, 133.2)
- added D15: APA102, gsg-modules:APA102-2020, F.Cu at (225.8, 138.6)
- added D150: APA102, gsg-modules:APA102-2020, F.Cu at (205.1, 154.2)
- added D151: APA102, gsg-modules:APA102-2020, F.Cu at (202.2, 156.9)
- added D152: APA102, gsg-modules:APA102-2020, F.Cu at (210.1, 148.8)
- added D153: APA102, gsg-modules:APA102-2020, F.Cu at (207.2, 151.5)
- added D154: APA102, gsg-modules:APA102-2020, F.Cu at (222.9, 135.2)
- added D155: APA102, gsg-modules:APA102-2020, F.Cu at (220.0, 137.9)
- added D156: APA102, gsg-modules:APA102-2020, F.Cu at (217.1, 140.7)
- added D157: APA102, gsg-modules:APA102-2020, F.Cu at (214.2, 143.4)
- added D158: APA102, gsg-modules:APA102-2020, F.Cu at (226.7, 130.5)
- added D159: APA102, gsg-modules:APA102-2020, F.Cu at (211.3, 146.1)
- added D16: APA102, gsg-modules:APA102-2020, F.Cu at (213.0, 151.5)
- added D160: APA102, gsg-modules:APA102-2020, F.Cu at (202.2, 154.2)
- added D161: APA102, gsg-modules:APA102-2020, F.Cu at (223.8, 132.5)
- added D162: APA102, gsg-modules:APA102-2020, F.Cu at (199.3, 156.9)
- added D163: APA102, gsg-modules:APA102-2020, F.Cu at (207.2, 148.8)
- added D164: APA102, gsg-modules:APA102-2020, F.Cu at (204.3, 151.5)
- added D165: APA102, gsg-modules:APA102-2020, F.Cu at (220.0, 135.2)
- added D166: APA102, gsg-modules:APA102-2020, F.Cu at (217.1, 138.0)
- added D167: APA102, gsg-modules:APA102-2020, F.Cu at (214.2, 140.7)
- added D168: APA102, gsg-modules:APA102-2020, F.Cu at (226.7, 127.8)
- added D169: APA102, gsg-modules:APA102-2020, F.Cu at (216.7, 154.2)
- added D17: APA102, gsg-modules:APA102-2020, F.Cu at (222.9, 140.6)
- added D170: APA102, gsg-modules:APA102-2020, F.Cu at (213.8, 156.9)
- added D171: APA102, gsg-modules:APA102-2020, F.Cu at (221.7, 148.7)
- added D172: APA102, gsg-modules:APA102-2020, F.Cu at (218.8, 151.5)
- added D173: APA102, gsg-modules:APA102-2020, F.Cu at (228.7, 141.3)
- added D174: APA102, gsg-modules:APA102-2020, F.Cu at (225.8, 144.0)
- added D175: APA102, gsg-modules:APA102-2020, F.Cu at (222.9, 146.0)
- added D176: APA102, gsg-modules:APA102-2020, F.Cu at (213.8, 154.2)
- added D177: APA102, gsg-modules:APA102-2020, F.Cu at (220.9, 132.5)
- added D178: APA102, gsg-modules:APA102-2020, F.Cu at (196.4, 156.9)
- added D179: APA102, gsg-modules:APA102-2020, F.Cu at (204.3, 148.8)
- added D18: APA102, gsg-modules:APA102-2020, F.Cu at (220.0, 143.3)
- added D180: APA102, gsg-modules:APA102-2020, F.Cu at (201.4, 151.5)
- added D181: APA102, gsg-modules:APA102-2020, F.Cu at (217.1, 135.3)
- added D182: APA102, gsg-modules:APA102-2020, F.Cu at (214.2, 138.0)
- added D183: APA102, gsg-modules:APA102-2020, F.Cu at (211.3, 140.7)
- added D184: APA102, gsg-modules:APA102-2020, F.Cu at (208.4, 143.4)
- added D185: APA102, gsg-modules:APA102-2020, F.Cu at (205.5, 146.0)
- added D186: APA102, gsg-modules:APA102-2020, F.Cu at (223.8, 127.1)
- added D187: APA102, gsg-modules:APA102-2020, F.Cu at (220.9, 129.8)
- added D188: APA102, gsg-modules:APA102-2020, F.Cu at (196.4, 154.2)
- added D189: APA102, gsg-modules:APA102-2020, F.Cu at (218.0, 132.5)
- added D19: APA102, gsg-modules:APA102-2020, F.Cu at (217.1, 146.1)
- added D190: APA102, gsg-modules:APA102-2020, F.Cu at (193.5, 156.9)
- added D191: APA102, gsg-modules:APA102-2020, F.Cu at (201.4, 148.8)
- added D192: APA102, gsg-modules:APA102-2020, F.Cu at (193.5, 154.2)
- added D193: APA102, gsg-modules:APA102-2020, F.Cu at (198.5, 151.5)
- added D194: APA102, gsg-modules:APA102-2020, F.Cu at (214.2, 135.3)
- added D195: APA102, gsg-modules:APA102-2020, F.Cu at (211.3, 138.0)
- added D196: APA102, gsg-modules:APA102-2020, F.Cu at (211.3, 143.4)
- added D197: APA102, gsg-modules:APA102-2020, F.Cu at (208.4, 146.1)
- added D198: APA102, gsg-modules:APA102-2020, F.Cu at (226.7, 125.1)
- added D199: APA102, gsg-modules:APA102-2020, F.Cu at (223.8, 129.8)
- added D2: APA102, gsg-modules:APA102-2020, F.Cu at (219.6, 156.9)
- added D20: APA102, gsg-modules:APA102-2020, F.Cu at (225.8, 135.9)
- added D200: APA102, gsg-modules:APA102-2020, F.Cu at (199.3, 154.2)
- added D21: APA102, gsg-modules:APA102-2020, F.Cu at (208.0, 154.2)
- added D22: APA102, gsg-modules:APA102-2020, F.Cu at (205.1, 156.9)
- added D23: APA102, gsg-modules:APA102-2020, F.Cu at (213.0, 148.8)
- added D24: APA102, gsg-modules:APA102-2020, F.Cu at (210.1, 151.5)
- added D25: APA102, gsg-modules:APA102-2020, F.Cu at (222.9, 137.9)
- added D26: APA102, gsg-modules:APA102-2020, F.Cu at (220.0, 140.6)
- added D27: APA102, gsg-modules:APA102-2020, F.Cu at (217.1, 143.4)
- added D28: APA102, gsg-modules:APA102-2020, F.Cu at (214.2, 146.1)
- added D29: APA102, gsg-modules:APA102-2020, F.Cu at (228.3, 157.5)
- added D3: APA102, gsg-modules:APA102-2020, F.Cu at (228.7, 146.7)
- added D30: APA102, gsg-modules:APA102-2020, F.Cu at (225.4, 157.5)
- added D31: APA102, gsg-modules:APA102-2020, F.Cu at (228.3, 154.8)
- added D32: APA102, gsg-modules:APA102-2020, F.Cu at (225.4, 154.8)
- added D33: APA102, gsg-modules:APA102-2020, F.Cu at (228.3, 152.1)
- added D34: APA102, gsg-modules:APA102-2020, F.Cu at (225.4, 152.1)
- added D35: APA102, gsg-modules:APA102-2020, F.Cu at (222.5, 156.8)
- added D36: APA102, gsg-modules:APA102-2020, F.Cu at (227.5, 149.4)
- added D37: APA102, gsg-modules:APA102-2020, F.Cu at (170.5, 89.2)
- added D38: APA102, gsg-modules:APA102-2020, F.Cu at (229.1, 92.1)
- added D39: APA102, gsg-modules:APA102-2020, F.Cu at (188.1, 139.4)
- added D4: APA102, gsg-modules:APA102-2020, F.Cu at (224.6, 149.4)
- added D40: APA102, gsg-modules:APA102-2020, F.Cu at (224.6, 102.9)
- added D41: APA102, gsg-modules:APA102-2020, F.Cu at (220.7, 108.2)
- added D42: APA102, gsg-modules:APA102-2020, F.Cu at (209.1, 119.1)
- added D43: APA102, gsg-modules:APA102-2020, F.Cu at (195.6, 135.3)
- added D44: APA102, gsg-modules:APA102-2020, F.Cu at (224.6, 105.6)
- added D45: APA102, gsg-modules:APA102-2020, F.Cu at (188.1, 142.1)
- added D46: APA102, gsg-modules:APA102-2020, F.Cu at (212.0, 119.1)
- added D47: APA102, gsg-modules:APA102-2020, F.Cu at (209.1, 121.8)
- added D48: APA102, gsg-modules:APA102-2020, F.Cu at (191.0, 140.6)
- added D49: APA102, gsg-modules:APA102-2020, F.Cu at (212.2, 127.2)
- added D5: APA102, gsg-modules:APA102-2020, F.Cu at (219.6, 154.2)
- added D50: APA102, gsg-modules:APA102-2020, F.Cu at (225.8, 111.6)
- added D51: APA102, gsg-modules:APA102-2020, F.Cu at (206.4, 132.5)
- added D52: APA102, gsg-modules:APA102-2020, F.Cu at (196.8, 140.7)
- added D53: APA102, gsg-modules:APA102-2020, F.Cu at (199.7, 138.0)
- added D54: APA102, gsg-modules:APA102-2020, F.Cu at (209.3, 127.2)
- added D55: APA102, gsg-modules:APA102-2020, F.Cu at (222.9, 116.3)
- added D56: APA102, gsg-modules:APA102-2020, F.Cu at (193.9, 143.3)
- added D57: APA102, gsg-modules:APA102-2020, F.Cu at (228.3, 108.9)
- added D58: APA102, gsg-modules:APA102-2020, F.Cu at (225.4, 108.9)
- added D59: APA102, gsg-modules:APA102-2020, F.Cu at (191.0, 146.0)
- added D6: APA102, gsg-modules:APA102-2020, F.Cu at (216.7, 156.9)
- added D60: APA102, gsg-modules:APA102-2020, F.Cu at (212.0, 124.5)
- added D61: APA102, gsg-modules:APA102-2020, F.Cu at (214.9, 121.8)
- added D62: APA102, gsg-modules:APA102-2020, F.Cu at (217.8, 119.0)
- added D63: APA102, gsg-modules:APA102-2020, F.Cu at (199.7, 140.7)
- added D64: APA102, gsg-modules:APA102-2020, F.Cu at (225.8, 114.3)
- added D65: APA102, gsg-modules:APA102-2020, F.Cu at (228.7, 111.6)
- added D66: APA102, gsg-modules:APA102-2020, F.Cu at (209.3, 132.6)
- added D67: APA102, gsg-modules:APA102-2020, F.Cu at (189.8, 151.4)
- added D68: APA102, gsg-modules:APA102-2020, F.Cu at (218.0, 127.1)
- added D69: APA102, gsg-modules:APA102-2020, F.Cu at (215.1, 129.9)
- added D7: APA102, gsg-modules:APA102-2020, F.Cu at (221.7, 151.4)
- added D70: APA102, gsg-modules:APA102-2020, F.Cu at (212.2, 132.6)
- added D71: APA102, gsg-modules:APA102-2020, F.Cu at (208.4, 135.3)
- added D72: APA102, gsg-modules:APA102-2020, F.Cu at (202.6, 140.7)
- added D73: APA102, gsg-modules:APA102-2020, F.Cu at (205.5, 137.9)
- added D74: APA102, gsg-modules:APA102-2020, F.Cu at (192.7, 151.4)
- added D75: APA102, gsg-modules:APA102-2020, F.Cu at (199.7, 143.4)
- added D76: APA102, gsg-modules:APA102-2020, F.Cu at (187.7, 155.6)
- added D77: APA102, gsg-modules:APA102-2020, F.Cu at (227.5, 106.2)
- added D78: APA102, gsg-modules:APA102-2020, F.Cu at (222.5, 110.9)
- added D79: APA102, gsg-modules:APA102-2020, F.Cu at (193.9, 140.6)
- added D8: APA102, gsg-modules:APA102-2020, F.Cu at (228.7, 144.0)
- added D80: APA102, gsg-modules:APA102-2020, F.Cu at (191.0, 143.3)
- added D81: APA102, gsg-modules:APA102-2020, F.Cu at (198.5, 135.3)
- added D82: APA102, gsg-modules:APA102-2020, F.Cu at (188.1, 144.8)
- added D83: APA102, gsg-modules:APA102-2020, F.Cu at (214.9, 119.1)
- added D84: APA102, gsg-modules:APA102-2020, F.Cu at (209.1, 124.5)
- added D85: APA102, gsg-modules:APA102-2020, F.Cu at (212.0, 121.8)
- added D86: APA102, gsg-modules:APA102-2020, F.Cu at (179.0, 155.5)
- added D87: APA102, gsg-modules:APA102-2020, F.Cu at (176.1, 155.5)
- added D88: APA102, gsg-modules:APA102-2020, F.Cu at (227.5, 103.5)
- added D89: APA102, gsg-modules:APA102-2020, F.Cu at (219.6, 110.9)
- added D9: APA102, gsg-modules:APA102-2020, F.Cu at (225.8, 146.7)
- added D90: APA102, gsg-modules:APA102-2020, F.Cu at (195.6, 151.5)
- added D91: APA102, gsg-modules:APA102-2020, F.Cu at (198.5, 148.8)
- added D92: APA102, gsg-modules:APA102-2020, F.Cu at (190.6, 156.8)
- added D93: APA102, gsg-modules:APA102-2020, F.Cu at (205.5, 140.6)
- added D94: APA102, gsg-modules:APA102-2020, F.Cu at (208.4, 138.0)
- added D95: APA102, gsg-modules:APA102-2020, F.Cu at (211.3, 135.3)
- added D96: APA102, gsg-modules:APA102-2020, F.Cu at (226.5, 119.7)
- added D97: APA102, gsg-modules:APA102-2020, F.Cu at (202.6, 143.4)
- added D98: APA102, gsg-modules:APA102-2020, F.Cu at (190.6, 154.1)
- added D99: APA102, gsg-modules:APA102-2020, F.Cu at (199.7, 146.1)
- added J1: TEST_1P, gsg-modules:TESTPOINT-50MIL, F.Cu at (95.4, 156.1)
- added J10: TEST_1P, gsg-modules:TESTPOINT-50MIL, F.Cu at (156.0, 156.1)
- added J11: TEST_1P, gsg-modules:TESTPOINT-50MIL, F.Cu at (159.5, 156.1)
- added J12: TEST_1P, gsg-modules:TESTPOINT-50MIL, F.Cu at (163.0, 157.9)
- added J13: TEST_1P, gsg-modules:TESTPOINT-50MIL, F.Cu at (166.5, 157.9)
- added J14: TEST_1P, gsg-modules:TESTPOINT-50MIL, F.Cu at (228.8, 97.1)
- added J15: TEST_1P, gsg-modules:TESTPOINT-50MIL, F.Cu at (228.8, 101.1)
- added J16: TEST_1P, gsg-modules:TESTPOINT-50MIL, F.Cu at (228.8, 99.1)
- added J17: TEST_1P, gsg-modules:TESTPOINT-50MIL, F.Cu at (132.6, 157.4)
- added J18: TEST_1P, gsg-modules:TESTPOINT-50MIL, F.Cu at (109.4, 156.1)
- added J19: TEST_1P, gsg-modules:TESTPOINT-50MIL, F.Cu at (98.9, 156.1)
- added J2: TEST_1P, gsg-modules:TESTPOINT-50MIL, F.Cu at (102.4, 156.1)
- added J20: TEST_1P, gsg-modules:TESTPOINT-50MIL, F.Cu at (91.9, 156.1)
- added J21: Conn_01x06, Pin_Headers:Pin_Header_Angled_1x06_Pitch1.27mm, F.Cu at (135.9, 67.3)
- added J22: USB_OTG, Connectors_USB:USB_Micro-B_Molex-105017-0001, F.Cu at (134.5, 135.5)
- added J23: Conn_01x02, Connectors_JST:JST_PH_S2B-PH-SM4-TB_02x2.00mm_Angled, F.Cu at (145.5, 108.0)
- added J24: Conn_01x06, Pin_Headers:Pin_Header_Angled_1x06_Pitch1.00mm, F.Cu at (135.9, 80.0)
- added J25: Conn_01x02, Connectors_JST:JST_PH_S2B-PH-SM4-TB_02x2.00mm_Angled, F.Cu at (119.4, 182.9)
- added J28: GS3, Connectors:GS3, F.Cu at (126.6, 152.7)
- added J29: TEST_1P, Measurement_Points:Measurement_Point_Round-SMD-Pad_Big, F.Cu at (194.2, 84.0)
- added J3: TEST_1P, gsg-modules:TESTPOINT-50MIL, F.Cu at (105.9, 156.1)
- added J30: TEST_1P, Measurement_Points:Measurement_Point_Round-SMD-Pad_Big, F.Cu at (163.2, 113.1)
- added J31: TEST_1P, Measurement_Points:Measurement_Point_Round-SMD-Pad_Big, F.Cu at (142.4, 134.5)
- added J32: TEST_1P, Measurement_Points:Measurement_Point_Round-SMD-Pad_Big, F.Cu at (182.4, 95.3)
- added J33: TEST_1P, Measurement_Points:Measurement_Point_Round-SMD-Pad_Big, F.Cu at (120.7, 154.7)
- added J4: TEST_1P, gsg-modules:TESTPOINT-50MIL, F.Cu at (125.7, 156.1)
- added J5: TEST_1P, gsg-modules:TESTPOINT-50MIL, F.Cu at (129.1, 157.4)
- added J6: TEST_1P, gsg-modules:TESTPOINT-50MIL, F.Cu at (136.1, 157.4)
- added J7: TEST_1P, gsg-modules:TESTPOINT-50MIL, F.Cu at (139.6, 157.4)
- added J8: TEST_1P, gsg-modules:TESTPOINT-50MIL, F.Cu at (152.5, 156.0)
- added J9: TEST_1P, gsg-modules:TESTPOINT-50MIL, F.Cu at (152.5, 158.0)
- added L1: Ferrite_Bead, Inductors_SMD:L_0805, F.Cu at (155.2, 109.9)
- added Q1: Q_NMOS_GDS, TO_SOT_Packages_SMD:SOT-89-3, F.Cu at (115.9, 146.4)
- added Q2: Q_NMOS_GDS, TO_SOT_Packages_SMD:SOT-89-3, F.Cu at (173.7, 95.5)
- added R1: R_Small, Resistors_SMD:R_0805, F.Cu at (175.0, 102.4)
- added R10: R, Resistors_SMD:R_0805, F.Cu at (205.9, 99.0)
- added R100: R, Resistors_SMD:R_0805, F.Cu at (187.8, 92.1)
- added R101: R, Resistors_SMD:R_0805, F.Cu at (161.9, 119.8)
- added R102: R, Resistors_SMD:R_0805, F.Cu at (199.6, 82.6)
- added R103: R, Resistors_SMD:R_0805, F.Cu at (138.5, 142.6)
- added R104: R, Resistors_SMD:R_0805, F.Cu at (194.9, 96.1)
- added R105: R, Resistors_SMD:R_0805, F.Cu at (146.3, 143.5)
- added R106: R, Resistors_SMD:R_0805, F.Cu at (178.6, 113.3)
- added R107: R, Resistors_SMD:R_0805, F.Cu at (203.8, 88.1)
- added R11: R, Resistors_SMD:R_0805, F.Cu at (186.0, 119.3)
- added R12: R, Resistors_SMD:R_0805, F.Cu at (210.5, 93.5)
- added R13: R, Resistors_SMD:R_0805, F.Cu at (175.1, 129.7)
- added R14: R, Resistors_SMD:R_0805, F.Cu at (214.8, 88.1)
- added R15: R_Small, Resistors_SMD:R_0805, F.Cu at (182.4, 102.0)
- added R16: R, Resistors_SMD:R_0805, F.Cu at (161.6, 141.6)
- added R17: R, Resistors_SMD:R_0805, F.Cu at (198.1, 104.4)
- added R18: R, Resistors_SMD:R_0805, F.Cu at (171.6, 129.7)
- added R19: R, Resistors_SMD:R_0805, F.Cu at (202.3, 99.0)
- added R2: R_Small, Resistors_SMD:R_0805, F.Cu at (133.2, 142.6)
- added R20: R, Resistors_SMD:R_0805, F.Cu at (182.5, 119.3)
- added R21: R, Resistors_SMD:R_0805, F.Cu at (192.4, 108.4)
- added R22: R, Resistors_SMD:R_0805, F.Cu at (153.8, 146.7)
- added R23: R, Resistors_SMD:R_0805, F.Cu at (168.0, 132.6)
- added R24: R, Resistors_SMD:R_0805, F.Cu at (145.4, 154.4)
- added R25: R, Resistors_SMD:R_0805, F.Cu at (158.1, 141.6)
- added R26: R, Resistors_SMD:R_0805, F.Cu at (217.7, 82.6)
- added R27: R, Resistors_SMD:R_0805, F.Cu at (207.0, 93.5)
- added R28: 0, Resistors_SMD:R_0805, F.Cu at (186.0, 113.9)
- added R29: R, Resistors_SMD:R_0805, F.Cu at (182.5, 113.9)
- added R3: 10k, Resistors_SMD:R_0805, F.Cu at (165.2, 138.0)
- added R30: R, Resistors_SMD:R_0805, F.Cu at (211.2, 88.1)
- added R31: R, Resistors_SMD:R_0805, F.Cu at (175.1, 124.2)
- added R32: R, Resistors_SMD:R_0805, F.Cu at (178.9, 118.8)
- added R33: 0, Resistors_SMD:R_0805, F.Cu at (149.5, 148.9)
- added R34: R, Resistors_SMD:R_0805, F.Cu at (192.8, 90.7)
- added R35: R, Resistors_SMD:R_0805, F.Cu at (131.2, 153.5)
- added R36: R, Resistors_SMD:R_0805, F.Cu at (187.4, 97.5)
- added R37: R, Resistors_SMD:R_0805, F.Cu at (142.4, 141.2)
- added R38: R, Resistors_SMD:R_0805, F.Cu at (168.3, 116.2)
- added R39: R, Resistors_SMD:R_0805, F.Cu at (138.2, 148.1)
- added R4: R, Resistors_SMD:R_0805, F.Cu at (153.1, 152.1)
- added R40: R, Resistors_SMD:R_0805, F.Cu at (161.6, 136.1)
- added R41: R, Resistors_SMD:R_0805, F.Cu at (198.8, 99.0)
- added R42: R, Resistors_SMD:R_0805, F.Cu at (188.9, 108.4)
- added R43: R, Resistors_SMD:R_0805, F.Cu at (194.5, 101.6)
- added R44: R, Resistors_SMD:R_0805, F.Cu at (171.6, 124.2)
- added R45: R, Resistors_SMD:R_0805, F.Cu at (203.4, 93.5)
- added R46: R, Resistors_SMD:R_0805, F.Cu at (214.1, 82.6)
- added R47: R, Resistors_SMD:R_0805, F.Cu at (158.1, 136.1)
- added R48: R, Resistors_SMD:R_0805, F.Cu at (207.7, 88.1)
- added R49: R, Resistors_SMD:R_0805, F.Cu at (154.5, 141.2)
- added R5: R, Resistors_SMD:R_0805, F.Cu at (157.3, 147.0)
- added R50: R, Resistors_SMD:R_0805, F.Cu at (185.3, 108.4)
- added R51: R, Resistors_SMD:R_0805, F.Cu at (168.0, 127.1)
- added R52: R, Resistors_SMD:R_0805, F.Cu at (146.0, 148.9)
- added R53: R, Resistors_SMD:R_0805, F.Cu at (164.5, 130.7)
- added R54: R, Resistors_SMD:R_0805, F.Cu at (141.9, 152.1)
- added R55: R, Resistors_SMD:R_0805, F.Cu at (190.9, 103.0)
- added R56: R, Resistors_SMD:R_0805, F.Cu at (175.4, 118.8)
- added R57: R, Resistors_SMD:R_0805, F.Cu at (150.2, 143.5)
- added R58: R, Resistors_SMD:R_0805, F.Cu at (210.6, 82.6)
- added R59: 0, Resistors_SMD:R_0805, F.Cu at (199.9, 93.5)
- added R6: R_Small, Resistors_SMD:R_0805, F.Cu at (153.4, 124.9)
- added R60: R, Resistors_SMD:R_0805, F.Cu at (171.8, 118.8)
- added R61: R, Resistors_SMD:R_0805, F.Cu at (138.3, 153.5)
- added R62: R, Resistors_SMD:R_0805, F.Cu at (154.5, 135.8)
- added R63: R, Resistors_SMD:R_0805, F.Cu at (189.6, 113.9)
- added R64: R, Resistors_SMD:R_0805, F.Cu at (221.2, 82.6)
- added R65: R, Resistors_SMD:R_0805, F.Cu at (149.0, 154.4)
- added R66: R, Resistors_SMD:R_0805, F.Cu at (178.7, 124.2)
- added R67: R, Resistors_SMD:R_0805, F.Cu at (199.9, 88.1)
- added R68: R, Resistors_SMD:R_0805, F.Cu at (160.9, 130.7)
- added R69: R, Resistors_SMD:R_0805, F.Cu at (187.4, 103.0)
- added R7: R_Small, Resistors_SMD:R_0805, F.Cu at (133.2, 148.1)
- added R70: R, Resistors_SMD:R_0805, F.Cu at (168.0, 121.7)
- added R71: R, Resistors_SMD:R_0805, F.Cu at (207.0, 82.6)
- added R72: R, Resistors_SMD:R_0805, F.Cu at (181.8, 107.4)
- added R73: R, Resistors_SMD:R_0805, F.Cu at (164.5, 125.2)
- added R74: R, Resistors_SMD:R_0805, F.Cu at (191.0, 97.5)
- added R75: R, Resistors_SMD:R_0805, F.Cu at (142.4, 146.6)
- added R76: R, Resistors_SMD:R_0805, F.Cu at (151.0, 138.0)
- added R77: R, Resistors_SMD:R_0805, F.Cu at (160.9, 125.2)
- added R78: R, Resistors_SMD:R_0805, F.Cu at (196.3, 90.7)
- added R79: R, Resistors_SMD:R_0805, F.Cu at (134.8, 153.5)
- added R8: R_Small, Resistors_SMD:R_0805, F.Cu at (169.7, 110.8)
- added R80: R, Resistors_SMD:R_0805, F.Cu at (189.6, 119.3)
- added R81: R, Resistors_SMD:R_0805, F.Cu at (165.2, 143.5)
- added R82: R, Resistors_SMD:R_0805, F.Cu at (178.7, 129.7)
- added R83: R, Resistors_SMD:R_0805, F.Cu at (209.4, 99.0)
- added R84: R, Resistors_SMD:R_0805, F.Cu at (224.8, 82.6)
- added R85: R, Resistors_SMD:R_0805, F.Cu at (214.1, 93.5)
- added R86: R, Resistors_SMD:R_0805, F.Cu at (160.9, 147.0)
- added R87: R, Resistors_SMD:R_0805, F.Cu at (196.7, 109.9)
- added R88: R, Resistors_SMD:R_0805, F.Cu at (218.3, 88.1)
- added R89: R, Resistors_SMD:R_0805, F.Cu at (193.1, 113.9)
- added R9: R_Small, Resistors_SMD:R_0805, F.Cu at (148.8, 132.6)
- added R90: R, Resistors_SMD:R_0805, F.Cu at (168.7, 138.0)
- added R91: R, Resistors_SMD:R_0805, F.Cu at (182.2, 124.8)
- added R92: R, Resistors_SMD:R_0805, F.Cu at (201.6, 104.4)
- added R93: R, Resistors_SMD:R_0805, F.Cu at (203.5, 82.6)
- added R94: R, Resistors_SMD:R_0805, F.Cu at (147.4, 138.0)
- added R95: R, Resistors_SMD:R_0805, F.Cu at (174.7, 113.3)
- added R96: R, Resistors_SMD:R_0805, F.Cu at (157.4, 130.3)
- added R97: R, Resistors_SMD:R_0805, F.Cu at (178.2, 107.9)
- added R98: R, Resistors_SMD:R_0805, F.Cu at (153.8, 130.3)
- added R99: R, Resistors_SMD:R_0805, F.Cu at (174.7, 107.9)
- added RV1: POT, Potentiometers:Potentiometer_Trimmer-EVM3S_R, F.Cu at (163.4, 104.2)
- added SW1: SW_Push, Buttons_Switches_SMD:SW_SPST_B3SL-1002P, F.Cu at (176.8, 85.5)
- added U1: 74AHCT1G125, TO_SOT_Packages_SMD:SOT-553, F.Cu at (155.7, 104.0)
- added U2: 74AHCT1G125, TO_SOT_Packages_SMD:SOT-553, F.Cu at (146.1, 117.1)
- added U3: S-8252_(SOT23), TO_SOT_Packages_SMD:SOT-23-6, F.Cu at (165.5, 83.9)
- added U4: MPU-6000, Housings_DFN_QFN:QFN-24_4x4mm_Pitch0.5mm_NoMask, F.Cu at (125.7, 145.9)
- added U5: L7805, TO_SOT_Packages_THT:TO-220-3_Horizontal, F.Cu at (47.0, 163.8)
- added U6: MTCH105, Housings_SSOP:TSSOP-14_4.4x5mm_Pitch0.65mm, F.Cu at (155.6, 117.6)
- added U7: STM32F407VGTx, Housings_QFP:LQFP-100_14x14mm_Pitch0.5mm, F.Cu at (68.6, 94.0)
- added U8: AZ1117-3.3, TO_SOT_Packages_SMD:SOT-223-3_TabPin2, F.Cu at (125.1, 136.0)
- added X1: Badgelife_shitty_connector, badgelife:Badgelife-Shitty-2x2, F.Cu at (76.2, 69.8)
- added Y1: Crystal, Crystals:Crystal_SMD_FOX_FE-2pin_7.5x5.0mm, F.Cu at (186.3, 84.7)

Commit message: Started placing components
Parts:
- J24: footprint Pin_Headers:Pin_Header_Angled_1x06_Pitch1.00mm -> Pin_Headers:Pin_Header_Angled_1x06_Pitch1.27mm
- moved X1 185.4 mm to (260.4, 48.3)
- moved C55 154.4 mm to (50.8, 94.0)
- moved R28 152.2 mm to (36.8, 83.8)
- moved C57 143.6 mm to (50.8, 88.9)
- moved R33 124.3 mm to (44.5, 82.5)
- moved J21 120.7 mm to (16.5, 85.1)
- moved J24 120.5 mm to (16.5, 96.5)
- moved J33 105.8 mm to (151.1, 53.3)
- moved L1 100.5 mm to (58.4, 82.5)
- moved U3 97.8 mm to (109.2, 163.8)
- moved Q2 85.3 mm to (128.3, 167.6)
- moved J22 81.9 mm to (68.6, 184.2)
- moved J23 75.7 mm to (134.6, 182.9)
- moved Y1 71.6 mm to (257.8, 86.4)
- moved J31 65.4 mm to (158.8, 71.1)
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
Commit message: Placing components wip, and fixing minor sch issues found along the way
Parts:
- added C71: C, Capacitors_SMD:C_0805, F.Cu at (256.8, 62.2)
- added R108: R, Resistors_SMD:R_0805, F.Cu at (268.0, 61.3)
- added R109: R, Resistors_SMD:R_0805, F.Cu at (271.1, 61.3)
- moved Y1 222.3 mm to (35.6, 91.4), turned to 90 degrees
- moved R12 187.3 mm to (28.3, 50.2)
- moved R26 184.1 mm to (36.5, 50.2)
- moved R30 183.3 mm to (34.0, 41.3), turned to 180 degrees
- moved R27 182.2 mm to (28.3, 57.8)
- moved R29 171.0 mm to (28.9, 38.7)
- moved R46 169.6 mm to (44.8, 91.4)
- moved R71 166.3 mm to (41.6, 99.1)
- moved R13 164.9 mm to (28.3, 54.6)
- moved R3 163.8 mm to (30.5, 44.8), turned to 90 degrees
- moved R19 160.8 mm to (41.6, 101.6), turned to 180 degrees
- moved R14 156.8 mm to (63.8, 45.7), turned to 180 degrees
- moved R84 153.9 mm to (71.1, 75.2), turned to 90 degrees
- moved R107 153.8 mm to (57.5, 40.6)
- moved R45 153.3 mm to (50.5, 82.5), turned to 180 degrees
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
Commit message: placed more components
Parts:
- moved C54 145.4 mm to (80.6, 83.8), turned to 90 degrees
- moved C51 129.4 mm to (57.1, 97.8), turned to 90 degrees
- moved R92 89.1 mm to (182.6, 48.9), turned to 180 degrees
- moved R22 85.7 mm to (108.9, 44.5), turned to 180 degrees
- moved R17 79.0 mm to (103.5, 164.2), turned to 90 degrees
- moved R26 62.1 mm to (86.0, 87.6), turned to 180 degrees
- moved R44 54.5 mm to (28.9, 33.7)
- moved R6 51.6 mm to (58.1, 55.2)
- moved R28 36.6 mm to (51.9, 89.9), turned to 180 degrees
- moved R94 34.5 mm to (78.1, 76.5), turned to 270 degrees
- moved R9 33.7 mm to (81.6, 50.2)
- moved L1 21.1 mm to (58.1, 103.5)
- moved R23 18.1 mm to (54.9, 101.0), turned to 180 degrees
- moved R88 17.6 mm to (86.0, 102.9)
- moved R100 15.3 mm to (43.2, 80.3)
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
Commit message: Started routing, and placed more components
Parts:
- moved C28 152.2 mm to (321.2, 117.9)
- moved C35 152.2 mm to (329.3, 107.7)
- moved C7 152.2 mm to (329.3, 113.0)
- moved C14 152.2 mm to (317.5, 110.3)
- moved C3 152.2 mm to (333.3, 107.7)
- moved C43 152.2 mm to (321.4, 112.6)
- moved C45 152.2 mm to (333.3, 113.0)
- moved C49 152.2 mm to (329.1, 118.3)
- moved C50 152.2 mm to (325.2, 118.3)
- moved C59 152.2 mm to (321.4, 107.3)
- moved C29 152.2 mm to (325.4, 113.0)
- moved C33 152.2 mm to (317.3, 121.1)
- moved C36 152.2 mm to (325.4, 107.7)
- moved C66 152.2 mm to (317.3, 115.8)
- moved C18 147.5 mm to (319.9, 100.7)
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Routing:
- net Net-(R31-Pad2): track 0.00 -> 43.7 mm, vias 0 -> 2
- net Net-(R14-Pad2): track 0.00 -> 23.7 mm, vias 0 -> 2
- net Net-(R79-Pad1): track 0.00 -> 20.1 mm
- net Net-(R19-Pad1): track 0.00 -> 19.9 mm
- net Net-(R73-Pad1): track 0.00 -> 19.4 mm
- net Net-(R20-Pad2): track 0.00 -> 17.0 mm
- net Net-(R75-Pad2): track 0.00 -> 16.6 mm
- net Net-(R18-Pad2): track 0.00 -> 16.4 mm
- net Net-(R71-Pad2): track 0.00 -> 16.0 mm
- net Net-(C51-Pad1): track 0.00 -> 14.7 mm
- net Net-(R26-Pad2): track 0.00 -> 14.0 mm
- net Net-(R89-Pad2): track 0.00 -> 12.8 mm
- net Net-(R34-Pad2): track 0.00 -> 12.7 mm
- net Net-(R61-Pad2): track 0.00 -> 12.4 mm
- net Net-(R33-Pad1): track 0.00 -> 11.7 mm
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
Commit message: Component placement madness
Parts:
- moved D38 133.4 mm to (210.0, 94.0)
- moved D29 107.7 mm to (174.0, 94.0)
- moved D30 102.1 mm to (178.0, 94.0)
- moved D26 101.4 mm to (162.0, 94.0)
- moved D31 99.6 mm to (182.0, 94.0)
- moved D101 97.9 mm to (162.0, 106.0)
- moved D27 96.6 mm to (166.0, 94.0)
- moved D77 94.6 mm to (166.0, 102.0)
- moved D32 94.2 mm to (186.0, 94.0)
- moved D176 92.3 mm to (162.0, 118.0)
- moved D28 92.1 mm to (170.0, 94.0)
- moved D33 91.6 mm to (190.0, 94.0)
- moved D102 91.6 mm to (166.0, 106.0)
- moved R22 89.2 mm to (197.5, 55.0), turned to 0 degrees
- moved D177 88.8 mm to (166.0, 118.0)
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Routing:
- net Net-(D8-Pad1): track 0.00 -> 2.30 mm
- net Net-(D7-Pad1): track 0.00 -> 2.30 mm
- net Net-(D6-Pad1): track 0.00 -> 2.30 mm
- net Net-(D5-Pad1): track 0.00 -> 2.30 mm
- net Net-(D4-Pad1): track 0.00 -> 2.30 mm
- net Net-(D3-Pad1): track 0.00 -> 2.30 mm
- net Net-(D23-Pad1): track 0.00 -> 2.30 mm
- net Net-(D22-Pad1): track 0.00 -> 2.30 mm
- net Net-(D21-Pad1): track 0.00 -> 2.30 mm
- net Net-(D2-Pad1): track 0.00 -> 2.30 mm
- net Net-(D19-Pad1): track 0.00 -> 2.30 mm
- net Net-(D18-Pad1): track 0.00 -> 2.30 mm
- net Net-(D17-Pad1): track 0.00 -> 2.30 mm
- net Net-(D16-Pad1): track 0.00 -> 2.30 mm
- net Net-(D15-Pad1): track 0.00 -> 2.30 mm
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
Commit message: Added script to wire up led data lines, and moved parts more
Parts:
- D1, D10, D100, D101, D102, D103, D104, D105, D106, D107, D108, D109, D11, D110, D111, D112, D113, D114, D115, D116, D117, D118, D119, D12, D120, D121, D122, D123, D124, D125, D126, D127, D128, D129, D13, D130, D131, D132, D133, D134, D135, D136, D137, D138, D139, D14, D140, D141, D142, D143, D144, D145, D146, D147, D148, D149, D15, D150, D151, D152, D153, D154, D155, D156, D157, D158, D159, D16, D160, D161, D162, D163, D164, D165, D166, D167, D168, D169, D17, D170, D171, D172, D173, D174, D175, D176, D177, D178, D179, D18, D180, D181, D182, D183, D184, D185, D186, D187, D188, D189, D19, D190, D191, D192, D193, D194, D195, D196, D197, D198, D199, D2, D20, D200, D21, D22, D23, D24, D25, D26, D27, D28, D29, D3, D30, D31, D32, D33, D34, D35, D36, D37, D38, D39, D4, D40, D41, D42, D43, D44, D45, D46, D47, D48, D49, D5, D50, D51, D52, D53, D54, D55, D56, D57, D58, D59, D6, D60, D61, D62, D63, D64, D65, D66, D67, D68, D69, D7, D70, D71, D72, D73, D74, D75, D76, D77, D78, D79, D8, D80, D81, D82, D83, D84, D85, D86, D87, D88, D89, D9, D90, D91, D92, D93, D94, D95, D96, D97, D98, D99: moved to B.Cu
- moved C53 57.6 mm to (335.1, 31.4)
- moved C12 57.6 mm to (322.6, 21.0)
- moved C15 57.6 mm to (325.9, 37.1)
- moved C2 57.6 mm to (339.7, 38.1)
- moved C21 57.6 mm to (326.0, 12.6)
- moved C22 57.6 mm to (336.4, -3.76)
- moved C29 57.6 mm to (330.5, 55.6)
- moved C36 57.6 mm to (330.5, 50.3)
- moved C66 57.6 mm to (322.4, 58.4)
- moved C1 57.6 mm to (338.4, 20.7)
- moved C10 57.6 mm to (339.3, 6.99)
- moved C16 57.6 mm to (332.1, 1.69)
- moved C17 57.6 mm to (342.8, -9.21)
- moved C24 57.6 mm to (321.0, 43.3)
- moved C27 57.6 mm to (336.8, 43.5)
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Routing:
- net Net-(D2-Pad6): track 0.00 -> 4.30 mm
- net Net-(D1-Pad6): track 0.00 -> 4.30 mm
- net Net-(D1-Pad1): track 0.00 -> 4.30 mm
- net Net-(D8-Pad1): track 2.30 -> 0.00 mm
- net Net-(D7-Pad1): track 2.30 -> 0.00 mm
- net Net-(D6-Pad1): track 2.30 -> 0.00 mm
- net Net-(D5-Pad1): track 2.30 -> 0.00 mm
- net Net-(D4-Pad1): track 2.30 -> 0.00 mm
- net Net-(D3-Pad1): track 2.30 -> 0.00 mm
- net Net-(D23-Pad1): track 2.30 -> 0.00 mm
- net Net-(D22-Pad1): track 2.30 -> 0.00 mm
- net Net-(D21-Pad1): track 2.30 -> 0.00 mm
- net Net-(D19-Pad1): track 2.30 -> 0.00 mm
- net Net-(D18-Pad1): track 2.30 -> 0.00 mm
- net Net-(D17-Pad1): track 2.30 -> 0.00 mm
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
Commit message: Fixed simple_wire.py and connected row data lines across
Routing:
- net Net-(D150-Pad6): track 0.00 -> 152.3 mm
- net Net-(D50-Pad1): track 0.00 -> 152.1 mm
- net Net-(D175-Pad6): track 0.00 -> 152.1 mm
- net /SCK100: track 0.00 -> 151.9 mm
- net Net-(D25-Pad6): track 0.00 -> 151.9 mm
- net Net-(D125-Pad6): track 0.00 -> 151.7 mm
- net Net-(D50-Pad6): track 0.00 -> 151.7 mm
- net Net-(D75-Pad6): track 0.00 -> 151.6 mm
- net /SDO100: track 0.00 -> 151.2 mm
- net Net-(D25-Pad1): track 0.00 -> 151.1 mm
- net Net-(D125-Pad1): track 0.00 -> 151.1 mm
- net Net-(D150-Pad1): track 0.00 -> 150.9 mm
- net Net-(D175-Pad1): track 0.00 -> 150.9 mm
- net Net-(D75-Pad1): track 0.00 -> 150.9 mm
- net Net-(D98-Pad6): track 0.00 -> 4.30 mm
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