File: ledbadge.kicad_pcb (KiCad board)
At the start: 4 copper layers, 426 parts, among them J1 TEST_1P, J10 TEST_1P, J11 TEST_1P, J12 TEST_1P, J13 TEST_1P, J14 TEST_1P, J15 TEST_1P, J16 TEST_1P, J17 TEST_1P, J18 TEST_1P, J19 TEST_1P, J2 TEST_1P, J20 TEST_1P, J21 Conn_01x06, J22 USB_OTG, J23 Conn_01x02, J24 Conn_01x06, J25 Conn_01x02, J28 GS3, J29 TEST_1P, J3 TEST_1P, J30 TEST_1P, J31 TEST_1P, J32 TEST_1P, J33 TEST_1P, J4 TEST_1P, J5 TEST_1P, J6 TEST_1P, J7 TEST_1P, J8 TEST_1P, J9 TEST_1P, Q1 Q_NMOS_GDS, Q2 Q_NMOS_GDS, SW1 SW_Push, U1 74AHCT1G125, U2 74AHCT1G125, U3 S-8252_(SOT23), U4 MPU-6000, U5 L7805, U6 MTCH105, U7 STM32F407VGTx, U8 AZ1117-3.3, X1 Badgelife_shitty_connector, Y1 Crystal

Commit message: Added board outline, placed more for 4layer layout
Parts:
- removed C71: C, Capacitors_SMD:C_0805
- removed R108, R109: R, Resistors_SMD:R_0805
- removed X1: Badgelife_shitty_connector, badgelife:Badgelife-Shitty-2x2
- C42: moved to B.Cu
- C47, C48: moved to F.Cu
- moved J10 248.6 mm to (360.8, 67.4)
- moved J5 248.6 mm to (359.8, 68.8)
- moved J12 248.2 mm to (360.3, 75.4)
- moved J17 248.2 mm to (361.8, 74.1)
- moved J14 226.7 mm to (369.3, 67.7)
- moved J19 226.7 mm to (369.1, 65.0)
- moved J2 225.8 mm to (367.9, 78.5)
- moved J7 225.8 mm to (369.4, 77.1)
- moved C14 180.5 mm to (244.9, 85.1)
- moved J4 165.9 mm to (333.0, 74.7)
- moved J11 165.9 mm to (339.9, 76.5)
- moved J16 165.9 mm to (341.4, 75.5)
- moved J9 165.9 mm to (333.6, 76.6)
- moved J20 151.3 mm to (394.8, 77.2)
- moved J15 151.3 mm to (396.1, 79.2)
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Routing:
- net +BATT: track 14.0 -> 61.8 mm
- net /USART1_RX: track 38.8 -> 0.00 mm, vias 2 -> 0
- net /NRST: track 29.6 -> 1.43 mm, vias 2 -> 0
- net +5V: track 0.00 -> 20.6 mm
- net Net-(J23-Pad2): track 42.2 -> 26.4 mm
- net Net-(C43-Pad2): track 15.8 -> 0.00 mm
- net Net-(R56-Pad2): track 0.00 -> 11.0 mm
- net +3V3: track 11.4 -> 21.8 mm, vias 0 -> 1
- net Net-(C44-Pad1): track 3.18 -> 11.4 mm
- net Net-(C64-Pad1): track 0.00 -> 8.21 mm
- net Net-(R18-Pad2): track 16.4 -> 24.5 mm, vias 0 -> 2
- net Net-(R107-Pad2): track 7.67 -> 0.00 mm
- net /MOSI_5v_R: track 0.00 -> 7.58 mm, vias 0 -> 1
- net Net-(R19-Pad1): track 19.9 -> 27.3 mm, vias 0 -> 2
- net Net-(R20-Pad2): track 17.0 -> 24.4 mm, vias 0 -> 2
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- added copper zone on F.Cu, net Net-(C43-Pad2)
- added copper zone on F.Cu, net Net-(Q1-Pad2)
Other:
- board outline added: 165.1 x 76.2 mm

Commit message: Moved LED clk and data traces to prevent SI issues
Parts:
- moved R25 17.4 mm to (103.1, 105.7), turned to 90 degrees
- moved R24 16.3 mm to (102.1, 102.1), turned to 270 degrees
- moved C43 7.62 mm to (151.4, 115.6)
- moved C44 7.62 mm to (154.9, 118.4)
- moved J23 7.62 mm to (141.6, 124.6)
- moved Q1 7.62 mm to (171.2, 114.9)
- moved Q2 7.62 mm to (177.2, 114.9)
- moved R5 7.62 mm to (152.4, 122.9)
- moved U3 7.62 mm to (154.9, 114.3)
- moved J25 7.62 mm to (170.8, 124.6)
- moved R17 7.62 mm to (151.3, 113.2)
- moved R4 7.62 mm to (162.3, 112.3)
- moved R21 4.90 mm to (98.6, 105.7)
- moved R22 2.41 mm to (100.8, 105.6)
Routing:
- net Net-(R25-Pad2): track 0.00 -> 11.1 mm
- net Net-(R24-Pad1): track 0.00 -> 7.51 mm
- net Net-(R21-Pad1): track 6.97 -> 0.00 mm
- net Net-(D23-Pad6): track 4.30 -> 0.00 mm
- net +BATT: track 61.8 -> 65.8 mm
- net Net-(J23-Pad2): track 26.4 -> 23.5 mm
- net /SCLK_3v3: track 2.33 -> 0.00 mm
- net /MOSI_3v3: track 2.23 -> 0.00 mm
- net Net-(R22-Pad2): track 10.3 -> 11.4 mm
- net Net-(R31-Pad2): track 39.2 -> 39.7 mm
- added copper zone on F.Cu, net GND

Commit message: Routed touch det signals, moved touchIC
Parts:
- moved RV1 75.5 mm to (121.0, 129.0)
- moved C70 73.6 mm to (109.0, 129.5)
- moved R92 69.7 mm to (114.0, 126.0), turned to 180 degrees
- moved R101 69.6 mm to (114.0, 115.0), turned to 270 degrees
- moved R37 59.9 mm to (121.2, 120.0), turned to 180 degrees
- moved J29 57.8 mm to (97.0, 114.8)
- moved J30 57.8 mm to (97.0, 118.0)
- moved J31 57.8 mm to (97.0, 123.1)
- moved J32 57.8 mm to (97.0, 126.2)
- moved J33 57.8 mm to (97.0, 120.5)
- moved R41 57.8 mm to (111.1, 114.7)
- moved R59 57.8 mm to (114.1, 129.4)
- moved U6 57.8 mm to (112.9, 119.9)
- moved R64 57.8 mm to (103.0, 114.8)
- moved R65 57.8 mm to (103.0, 118.0)
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Routing:
- net /~TOUCH4_DET: track 4.56 -> 64.4 mm, vias 0 -> 2
- net /~TOUCH3_DET: track 6.79 -> 64.7 mm, vias 0 -> 2
- net /~TOUCH1_DET: track 6.53 -> 62.3 mm, vias 0 -> 2
- net /~TOUCH0_DET: track 3.94 -> 56.8 mm, vias 0 -> 2
- net +5V: track 20.6 -> 57.6 mm, vias 0 -> 20
- net /MOSI_3v3: track 0.00 -> 22.2 mm
- net /SCLK_3v3: track 0.00 -> 21.7 mm
- net /SENSITIVITY_ADJ: track 0.00 -> 17.9 mm
- net /DAC_OUT1: track 0.00 -> 16.8 mm
- net /SERIAL_TXO: track 0.00 -> 10.7 mm
- net /SERIAL_PWR: track 0.00 -> 7.99 mm
- net /SERIAL_RXI: track 0.00 -> 7.24 mm
- net Net-(R92-Pad1): track 0.00 -> 5.55 mm
- net /~TOUCH2/GC: track 11.7 -> 9.49 mm
- added copper zone on In2.Cu, net +5V
- added copper zone on B.Cu, net GND

Commit message: Setup more copper layers, routed power and ground
Parts:
- C14, C15: moved to B.Cu
- moved C35 322.7 mm to (50.0, 89.3)
- moved C36 322.7 mm to (46.0, 89.3)
- moved C52 284.0 mm to (97.5, 94.8), turned to 225 degrees
- moved C45 282.9 mm to (94.8, 98.0), turned to 180 degrees
- moved C56 222.3 mm to (164.2, 76.8), turned to 90 degrees
- moved C40 162.4 mm to (212.4, 38.3)
- moved C41 162.4 mm to (217.1, 32.8)
- moved C37 153.6 mm to (214.8, 43.8)
- moved C38 123.7 mm to (223.2, 42.8)
- moved C15 117.2 mm to (129.8, 67.2)
- moved C14 85.9 mm to (160.8, 67.8)
- moved J1 77.5 mm to (363.0, 90.8)
- moved J6 77.5 mm to (363.0, 89.0)
- moved J22 7.19 mm to (229.3, 113.5)
- moved Q2 5.15 mm to (182.3, 114.2), turned to 180 degrees
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Routing:
- net /ACCEL_INT: track 0.00 -> 87.9 mm, vias 0 -> 2
- net /SCL: track 0.00 -> 77.4 mm, vias 0 -> 2
- net /SDA: track 0.00 -> 74.4 mm, vias 0 -> 2
- net +5V: track 57.6 -> 104.5 mm, vias 20 -> 30
- net +3V3: track 21.8 -> 64.2 mm, vias 1 -> 23
- net /NRST: track 1.43 -> 41.6 mm, vias 0 -> 2
- net /SWO: track 0.00 -> 40.0 mm, vias 0 -> 2
- net /USART1_RX: track 0.00 -> 38.0 mm
- net Net-(Q2-Pad1): track 0.00 -> 35.4 mm
- net /USB_VBUS: track 0.00 -> 31.8 mm
- net /SWCLK: track 0.00 -> 19.5 mm
- net Net-(Q1-Pad1): track 0.00 -> 14.3 mm
- net /SWDIO: track 0.00 -> 12.5 mm
- net Net-(C64-Pad1): track 8.21 -> 16.9 mm
- net Net-(Q1-Pad2): track 6.00 -> 0.00 mm
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- added copper zone on In1.Cu, net +3V3

Commit message: More routing completed
Parts:
- removed C37, C40: C, Capacitors_SMD:C_0805
- removed J1, J10, J11, J12, J13, J14, J15, J16, J17, J18, J19, J2, J20, J3, J4, J5, J6, J7, J8, J9: TEST_1P, gsg-modules:TESTPOINT-50MIL
- C35, C36, C38: moved to B.Cu
- moved C38 123.0 mm to (105.8, 79.0), turned to 0 degrees
- moved C41 122.3 mm to (109.5, 91.0), turned to 180 degrees
- moved C36 61.5 mm to (107.0, 97.5), turned to 180 degrees
- moved C35 59.7 mm to (109.5, 85.0)
- moved C47 4.16 mm to (94.8, 98.0), turned to 180 degrees
- moved R21 3.59 mm to (99.5, 102.2)
- moved L1 2.61 mm to (97.8, 99.0)
- moved C45 2.00 mm to (94.8, 100.0)
- moved SW1 1.41 mm to (82.0, 78.2), turned to 180 degrees
Routing:
- net +5V: track 104.5 -> 217.9 mm, vias 30 -> 63
- net +3V3: track 64.2 -> 112.4 mm, vias 23 -> 40
- net /NRST: track 41.6 -> 69.4 mm, vias 2 -> 4
- net Net-(R21-Pad1): track 0.00 -> 7.85 mm
- net /VDDA: track 9.63 -> 10.8 mm
Other:
- net class Default: clearance 0.2 -> 0.127; trace_width 0.25 -> 0.127; via_dia 0.6 -> 0.3556; via_drill 0.4 -> 0.254
- rule trace_clearance: 0.2 -> 0.127
- rule trace_min: 0.2 -> 0.127
- rule via_min_drill: 0.3 -> 0.254
- rule via_min_size: 0.4 -> 0.3556

Commit message: Added more vias for LED power
Routing:
- net +5V: track 217.9 -> 223.4 mm, vias 63 -> 67
Changed lines of the file:
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@@
     (links 1154)
     (no_connects 166)
-    (area 65.964999 55.804999 233.865 132.155001)
+    (area 65.964999 55.804999 233.792 132.155001)
     (thickness 1.6)
     (drawings 5)
-    (tracks 1587)
+    (tracks 1601)
     (zones 0)
     (modules 400)
@@
   (page A4)
   (layers
-    (0 F.Cu signal)
-    (1 In1.Cu signal)
+    (0 F.Cu signal hide)
+    (1 In1.Cu signal hide)
     (2 In2.Cu signal hide)
     (31 B.Cu signal)
@@
     (pad_to_mask_clearance 0.2)
     (aux_axis_origin 0 0)
-    (visible_elements FFFEFFFF)
+    (visible_elements FFFEBFFF)
     (pcbplotparams
       (layerselection 0x00030_80000001)
@@
   (gr_line (start 231.14 55.88) (end 231.14 132.08) (layer Edge.Cuts) (width 0.15))
   (gr_line (start 66.04 55.88) (end 228.6 55.88) (layer Edge.Cuts) (width 0.15))
+  (segment (start 113.109 81.638194) (end 113.861806 81.638194) (width 0.127) (layer B.Cu) (net 1))
+  (segment (start 113.861806 81.638194) (end 114 81.5) (width 0.127) (layer B.Cu) (net 1))
+  (via (at 114 81.5) (size 0.3556) (drill 0.254) (layers F.Cu B.Cu) (net 1))
+  (segment (start 107.109 81.638194) (end 107.861806 81.638194) (width 0.127) (layer B.Cu) (net 1))
+  (segment (start 107.861806 81.638194) (end 107.989586 81.510414) (width 0.127) (layer B.Cu) (net 1))
+  (via (at 107.989586 81.510414) (size 0.3556) (drill 0.254) (layers F.Cu B.Cu) (net 1))
+  (segment (start 100.917 79.846) (end 100.917 78.917) (width 0.127) (layer B.Cu) (net 1))
+  (segment (start 100.917 78.917) (end 100.9 78.9) (width 0.127) (layer B.Cu) (net 1))
+  (via (at 100.9 78.9) (size 0.3556) (drill 0.254) (layers F.Cu B.Cu) (net 1))
+  (segment (start 101.109 81.638194) (end 101.109 80.038) (width 0.127) (layer B.Cu) (net 1))
+  (segment (start 101.109 80.038) (end 100.917 79.846) (width 0.127) (layer B.Cu) (net 1))
+  (segment (start 77.109 81.638194) (end 77.109 81.109) (width 0.127) (layer B.Cu) (net 1))
+  (segment (start 77.109 81.109) (end 76.9 80.9) (width 0.127) (layer B.Cu) (net 1))
+  (via (at 76.9 80.9) (size 0.3556) (drill 0.254) (layers F.Cu B.Cu) (net 1))
   (segment (start 95.109 81.638194) (end 95.168 81.638194) (width 0.25) (layer B.Cu) (net 1))
   (segment (start 95.168 81.638194) (end 95.8 81.006194) (width 0.25) (layer B.Cu) (net 1))

Commit message: more vias
Routing:
- net +5V: track 223.4 -> 283.4 mm, vias 67 -> 109

Commit message: Added more vias
Routing:
- net +5V: track 283.4 -> 302.2 mm, vias 109 -> 125
