File: ledbadge.kicad_pcb (KiCad board)
At the start: 4 copper layers, 165.1 x 76.2 mm, 400 parts, among them J21 Conn_01x06, J22 USB_OTG, J23 Conn_01x02, J24 Conn_01x06, J25 Conn_01x02, J28 GS3, J29 TEST_1P, J30 TEST_1P, J31 TEST_1P, J32 TEST_1P, J33 TEST_1P, Q1 Q_NMOS_GDS, Q2 Q_NMOS_GDS, SW1 SW_Push, U1 74AHCT1G125, U2 74AHCT1G125, U3 S-8252_(SOT23), U4 MPU-6000, U5 L7805, U6 MTCH105, U7 STM32F407VGTx, U8 AZ1117-3.3, Y1 Crystal

Commit message: Added all the LED 5V vias
Parts:
- moved C32 0.55 mm to (220.2, 103.8)
Routing:
- net +5V: track 302.2 -> 373.4 mm, vias 125 -> 185

Commit message: Fixed DRC for via-trace distance
Parts:
- moved J28 13.3 mm to (212.6, 104.0)
Routing:
- net /USB_VBUS: track 31.8 -> 18.2 mm
- net Net-(C64-Pad1): track 16.9 -> 29.9 mm
- net +5V: track 373.4 -> 371.0 mm, vias 185 -> 189
- net Net-(J23-Pad2): track 23.5 -> 25.1 mm

Commit message: Fixing DRC and unconnected nets
Connections:
- C61 pad 1: +5V -> Net-(C61-Pad1)
- C62 pad 1: +5V -> Net-(C61-Pad1)
- C63 pad 1: +5V -> Net-(C61-Pad1)
- C64 pad 1: Net-(C64-Pad1) -> +5V
- C65 pad 1: Net-(C64-Pad1) -> +5V
- C66 pad 1: Net-(C64-Pad1) -> +5V
- J28 pad 1: +5V -> Net-(C61-Pad1)
- J28 pad 2: Net-(C64-Pad1) -> +5V
- U5 pad 3: +5V -> Net-(C61-Pad1)
- U8 pad 3: Net-(C64-Pad1) -> +5V
Routing:
- net +5V: track 371.0 -> 401.0 mm, vias 189 -> 202
- net Net-(C64-Pad1): track 29.9 -> 0.00 mm
- net Net-(C61-Pad1): track 0.00 -> 23.7 mm

Commit message: Added touchpads and guard
Routing:
- net Net-(J32-Pad1): track 5.09 -> 118.4 mm, vias 0 -> 1
- net Net-(J31-Pad1): track 5.09 -> 70.8 mm, vias 0 -> 1
- net /~TOUCH2/GC: track 9.49 -> 67.4 mm, vias 0 -> 2
- net GND: track 0.28 -> 37.7 mm
- net Net-(J30-Pad1): track 5.09 -> 31.1 mm, vias 0 -> 1
- net Net-(J29-Pad1): track 5.09 -> 15.7 mm, vias 0 -> 1
- net +5V: track 401.0 -> 393.2 mm, vias 202 -> 207
- net Net-(Q2-Pad1): track 35.4 -> 34.1 mm
- net /TOUCH2/GUARD: vias 0 -> 1
- added copper zone on In2.Cu, net /TOUCH2/GUARD
- added copper zone on B.Cu, net Net-(J29-Pad1)
- added copper zone on B.Cu, net Net-(J30-Pad1)
- added copper zone on B.Cu, net Net-(J31-Pad1)
- added copper zone on B.Cu, net Net-(J32-Pad1)
Other:
- rule pad_to_mask_clearance: 0.2 -> 0.0508

Commit message: Layout tweaks
Parts:
- moved J22 9.51 mm to (229.3, 104.0)
Routing:
- net +5V: track 393.2 -> 399.2 mm, vias 207 -> 206
- net /USB_VBUS: track 18.2 -> 13.8 mm
- net GND: track 37.7 -> 39.4 mm
Changed lines of the file:
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@@
   (general
     (links 1154)
-    (no_connects 10)
+    (no_connects 11)
     (area 65.9 55.804999 233.792 132.155001)
     (thickness 1.6)
     (drawings 5)
-    (tracks 2144)
+    (tracks 2146)
     (zones 0)
     (modules 400)
@@
   (layers
     (0 F.Cu signal)
-    (1 In1.Cu signal hide)
+    (1 In1.Cu signal)
     (2 In2.Cu signal)
     (31 B.Cu signal)
@@
   )
   (setup
-    (last_trace_width 0.127)
-    (user_trace_width 0.25)
+    (last_trace_width 0.25)
     (user_trace_width 0.25)
+    (user_trace_width 0.5)
+    (user_trace_width 0.75)
     (user_trace_width 1)
     (user_trace_width 1.5)
     (user_trace_width 2)
-    (user_trace_width 5)
+    (user_trace_width 2.5)
     (trace_clearance 0.127)
     (zone_clearance 0.127)
@@
   )
   (module Connectors_USB:USB_Micro-B_Molex-105017-0001 (layer F.Cu)
-    (at 229.34 113.51 90)
+    (at 229.34 104 90)
     (descr http://www.molex.com/pdm_docs/sd/1050170001_sd.pdf)
     (tags "Micro-USB SMD Typ-B")
@@
   (gr_line (start 231.14 55.88) (end 231.14 132.08) (layer Edge.Cuts) (width 0.15))
   (gr_line (start 66.04 55.88) (end 228.6 55.88) (layer Edge.Cuts) (width 0.15))
+  (segment (start 79.6 111.8) (end 79.6 110.3) (width 0.25) (layer F.Cu) (net 1))
+  (segment (start 79.6 110.3) (end 81.4 108.5) (width 0.25) (layer F.Cu) (net 1))
+  (segment (start 82.268 112.346194) (end 80.146194 112.346194) (width 0.25) (layer F.Cu) (net 1))
+  (segment (start 80.146194 112.346194) (end 79.6 111.8) (width 0.25) (layer F.Cu) (net 1))
   (segment (start 100.9 67.8) (end 101.9 67.8) (width 0.25) (layer B.Cu) (net 1))
   (via (at 101.9 67.8) (size 0.3556) (drill 0.254) (layers F.Cu B.Cu) (net 1))
@@
   (via (at 84.1 87.2) (size 0.3556) (drill 0.254) (layers F.Cu B.Cu) (net 1))
   (segment (start 83.661806 87.638194) (end 84.1 87.2) (width 0.127) (layer B.Cu) (net 1))
-  (segment (start 82.268 112.346194) (end 81.453806 112.346194) (width 0.127) (layer F.Cu) (net 1))
-  (segment (start 81.453806 112.346194) (end 81.4 112.4) (width 0.127) (layer F.Cu) (net 1))
-  (via (at 81.4 112.4) (size 0.3556) (drill 0.254) (layers F.Cu B.Cu) (net 1))
   (segment (start 82.239809 108.492194) (end 81.407806 108.492194) (width 0.127) (layer F.Cu) (net 1))
   (segment (start 81.407806 108.492194) (end 81.4 108.5) (width 0.127) (layer F.Cu) (net 1))
@@
   (segment (start 204.331 84.059) (end 204.331 86.551) (width 1) (layer F.Cu) (net 1))
   (segment (start 204.331 86.551) (end 204.027 86.855) (width 1) (layer F.Cu) (net 1))
+  (segment (start 226.99 102.7) (end 225.3 102.7) (width 0.5) (layer F.Cu) (net 2))
   (segment (start 183 110.6) (end 183.4 110.6) (width 0.127) (layer F.Cu) (net 2))
   (segment (start 165.9 110.6) (end 183 110.6) (width 0.127) (layer F.Cu) (net 2))
@@
   (segment (start 128.358804 67.274999) (end 129.75 68.666195) (width 0.25) (layer F.Cu) (net 423))
   (via (at 129.75 68.666195) (size 0.3556) (drill 0.254) (layers F.Cu B.Cu) (net 423))
-  (segment (start 225.8 114.8) (end 225.81 114.81) (width 0.5) (layer F.Cu) (net 425))
-  (segment (start 225.81 114.81) (end 226.99 114.81) (width 0.5) (layer F.Cu) (net 425))
-  (segment (start 224.52 114.8) (end 225.8 114.8) (width 1) (layer F.Cu) (net 425))
+  (segment (start 225.8 105.3) (end 226.99 105.3) (width 0.5) (layer F.Cu) (net 425))
+  (segment (start 224.495199 103.995199) (end 225.8 105.3) (width 1) (layer F.Cu) (net 425))
+  (segment (start 213.87 104) (end 220.608894 104) (width 1) (layer F.Cu) (net 425))
+  (segment (start 220.608894 104) (end 220.613695 103.995199) (width 1) (layer F.Cu) (net 425))
+  (segment (start 220.613695 103.995199) (end 224.495199 103.995199) (width 1) (layer F.Cu) (net 425))
   (segment (start 213.87 104) (end 213.87 104.15) (width 1) (layer F.Cu) (net 425))
-  (segment (start 213.87 104.15) (end 224.52 114.8) (width 1) (layer F.Cu) (net 425))
-  (segment (start 226.450998 114.81) (end 226.99 114.81) (width 0.5) (layer F.Cu) (net 425))
   (segment (start 165.145 125.581) (end 152.4 125.581) (width 1) (layer F.Cu) (net 428))
   (segment (start 152.4 125.581) (end 144.445 125.581) (width 1) (layer F.Cu) (net 428))

Commit message: Tweaked some footprints
Routing:
- net Net-(J32-Pad1): track 118.4 -> 116.2 mm
- net Net-(J31-Pad1): track 70.8 -> 72.3 mm
Changed lines of the file:
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@@
   (general
     (links 1154)
-    (no_connects 11)
+    (no_connects 8)
     (area 65.9 55.804999 233.792 132.155001)
     (thickness 1.6)
     (drawings 5)
-    (tracks 2146)
+    (tracks 2148)
     (zones 0)
     (modules 400)
@@
   (layers
     (0 F.Cu signal)
-    (1 In1.Cu signal)
-    (2 In2.Cu signal)
-    (31 B.Cu signal)
+    (1 In1.Cu signal hide)
+    (2 In2.Cu signal hide)
+    (31 B.Cu signal hide)
     (32 B.Adhes user)
     (33 F.Adhes user hide)
@@
     (pad_to_mask_clearance 0.0508)
     (aux_axis_origin 0 0)
-    (visible_elements FFFEFFFF)
+    (visible_elements FFFE7FFF)
     (pcbplotparams
       (layerselection 0x00030_80000001)
@@
     (add_net "Net-(U7-Pad91)")
   )
+  (module TO_SOT_Packages_THT:TO-220-3_Horizontal (layer F.Cu)
+    (at 196.446 109.22 270)
+    (descr "TO-220-3, Horizontal, RM 2.54mm")
+    (tags "TO-220-3 Horizontal RM 2.54mm")
+    (fp_text reference U5 (at 2.54 -20.58 270) (layer F.SilkS)
+      (effects (font (size 1 1) (thickness 0.15)))
+    )
+    (fp_text value L7805 (at 2.54 1.9 270) (layer F.Fab)
+      (effects (font (size 1 1) (thickness 0.15)))
+    )
+    (fp_text user %R (at 2.54 -20.58 270) (layer F.Fab)
+      (effects (font (size 1 1) (thickness 0.15)))
+    )
+    (fp_line (start -2.46 -13.06) (end -2.46 -19.46) (layer F.Fab) (width 0.1))
+    (fp_line (start -2.46 -19.46) (end 7.54 -19.46) (layer F.Fab) (width 0.1))
+    (fp_line (start 7.54 -19.46) (end 7.54 -13.06) (layer F.Fab) (width 0.1))
+    (fp_line (start 7.54 -13.06) (end -2.46 -13.06) (layer F.Fab) (width 0.1))
+    (fp_line (start -2.46 -3.81) (end -2.46 -13.06) (layer F.Fab) (width 0.1))
+    (fp_line (start -2.46 -13.06) (end 7.54 -13.06) (layer F.Fab) (width 0.1))
+    (fp_line (start 7.54 -13.06) (end 7.54 -3.81) (layer F.Fab) (width 0.1))
+    (fp_line (start 7.54 -3.81) (end -2.46 -3.81) (layer F.Fab) (width 0.1))
+    (fp_line (start 0 -3.81) (end 0 0) (layer F.Fab) (width 0.1))
+    (fp_line (start 2.54 -3.81) (end 2.54 0) (layer F.Fab) (width 0.1))
+    (fp_line (start 5.08 -3.81) (end 5.08 0) (layer F.Fab) (width 0.1))
+    (fp_line (start -2.58 -3.69) (end 7.66 -3.69) (layer F.SilkS) (width 0.12))
+    (fp_line (start -2.58 -19.58) (end 7.66 -19.58) (layer F.SilkS) (width 0.12))
+    (fp_line (start -2.58 -19.58) (end -2.58 -3.69) (layer F.SilkS) (width 0.12))
+    (fp_line (start 7.66 -19.58) (end 7.66 -3.69) (layer F.SilkS) (width 0.12))
+    (fp_line (start 0 -3.69) (end 0 -1.05) (layer F.SilkS) (width 0.12))
+    (fp_line (start 2.54 -3.69) (end 2.54 -1.066) (layer F.SilkS) (width 0.12))
+    (fp_line (start 5.08 -3.69) (end 5.08 -1.066) (layer F.SilkS) (width 0.12))
+    (fp_line (start -2.71 -19.71) (end -2.71 1.15) (layer F.CrtYd) (width 0.05))
+    (fp_line (start -2.71 1.15) (end 7.79 1.15) (layer F.CrtYd) (width 0.05))
+    (fp_line (start 7.79 1.15) (end 7.79 -19.71) (layer F.CrtYd) (width 0.05))
+    (fp_line (start 7.79 -19.71) (end -2.71 -19.71) (layer F.CrtYd) (width 0.05))
+    (pad 1 thru_hole rect (at 0 0 270) (size 1.8 1.8) (drill 1) (layers *.Cu *.Mask)
+      (net 15 +BATT))
+    (pad 2 thru_hole oval (at 2.54 0 270) (size 1.8 1.8) (drill 1) (layers *.Cu *.Mask)
+      (net 2 GND))
+    (pad 3 thru_hole oval (at 5.08 0 270) (size 1.8 1.8) (drill 1) (layers *.Cu *.Mask)
+      (net 606 "Net-(C61-Pad1)"))
+    (model ${KISYS3DMOD}/TO_SOT_Packages_THT.3dshapes/TO-220-3_Horizontal.wrl
+      (at (xyz 0.1 0 0))
+      (scale (xyz 0.393701 0.393701 0.393701))
+      (rotate (xyz 0 0 0))
+    )
+  )
   (module Crystals:Crystal_SMD_FOX_FE-2pin_7.5x5.0mm (layer F.Cu)
     (at 86.776 89.525194 270)
@@
     )
   )
-  (module TO_SOT_Packages_THT:TO-220-3_Horizontal (layer F.Cu)
-    (at 196.446 109.22 270)
-    (descr "TO-220-3, Horizontal, RM 2.54mm")
-    (tags "TO-220-3 Horizontal RM 2.54mm")
-    (fp_text reference U5 (at 2.54 -20.58 270) (layer F.SilkS)
-      (effects (font (size 1 1) (thickness 0.15)))
-    )
-    (fp_text value L7805 (at 2.54 1.9 270) (layer F.Fab)
-      (effects (font (size 1 1) (thickness 0.15)))
-    )
-    (fp_text user %R (at 2.54 -20.58 270) (layer F.Fab)
-      (effects (font (size 1 1) (thickness 0.15)))
-    )
-    (fp_line (start -2.46 -13.06) (end -2.46 -19.46) (layer F.Fab) (width 0.1))
-    (fp_line (start -2.46 -19.46) (end 7.54 -19.46) (layer F.Fab) (width 0.1))
-    (fp_line (start 7.54 -19.46) (end 7.54 -13.06) (layer F.Fab) (width 0.1))
-    (fp_line (start 7.54 -13.06) (end -2.46 -13.06) (layer F.Fab) (width 0.1))
-    (fp_line (start -2.46 -3.81) (end -2.46 -13.06) (layer F.Fab) (width 0.1))
-    (fp_line (start -2.46 -13.06) (end 7.54 -13.06) (layer F.Fab) (width 0.1))
-    (fp_line (start 7.54 -13.06) (end 7.54 -3.81) (layer F.Fab) (width 0.1))
-    (fp_line (start 7.54 -3.81) (end -2.46 -3.81) (layer F.Fab) (width 0.1))
-    (fp_line (start 0 -3.81) (end 0 0) (layer F.Fab) (width 0.1))
-    (fp_line (start 2.54 -3.81) (end 2.54 0) (layer F.Fab) (width 0.1))
-    (fp_line (start 5.08 -3.81) (end 5.08 0) (layer F.Fab) (width 0.1))
-    (fp_line (start -2.58 -3.69) (end 7.66 -3.69) (layer F.SilkS) (width 0.12))
-    (fp_line (start -2.58 -19.58) (end 7.66 -19.58) (layer F.SilkS) (width 0.12))
-    (fp_line (start -2.58 -19.58) (end -2.58 -3.69) (layer F.SilkS) (width 0.12))
-    (fp_line (start 7.66 -19.58) (end 7.66 -3.69) (layer F.SilkS) (width 0.12))
-    (fp_line (start 0 -3.69) (end 0 -1.05) (layer F.SilkS) (width 0.12))
-    (fp_line (start 2.54 -3.69) (end 2.54 -1.066) (layer F.SilkS) (width 0.12))
-    (fp_line (start 5.08 -3.69) (end 5.08 -1.066) (layer F.SilkS) (width 0.12))
-    (fp_line (start -2.71 -19.71) (end -2.71 1.15) (layer F.CrtYd) (width 0.05))
-    (fp_line (start -2.71 1.15) (end 7.79 1.15) (layer F.CrtYd) (width 0.05))
-    (fp_line (start 7.79 1.15) (end 7.79 -19.71) (layer F.CrtYd) (width 0.05))
-    (fp_line (start 7.79 -19.71) (end -2.71 -19.71) (layer F.CrtYd) (width 0.05))
-    (fp_circle (center 2.54 -16.66) (end 4.39 -16.66) (layer F.Fab) (width 0.1))
-    (pad 0 np_thru_hole oval (at 2.54 -16.66 270) (size 3.5 3.5) (drill 3.5) (layers *.Cu *.Mask))
-    (pad 1 thru_hole rect (at 0 0 270) (size 1.8 1.8) (drill 1) (layers *.Cu *.Mask)
-      (net 15 +BATT))
-    (pad 2 thru_hole oval (at 2.54 0 270) (size 1.8 1.8) (drill 1) (layers *.Cu *.Mask)
-      (net 2 GND))
-    (pad 3 thru_hole oval (at 5.08 0 270) (size 1.8 1.8) (drill 1) (layers *.Cu *.Mask)
-      (net 606 "Net-(C61-Pad1)"))
-    (model ${KISYS3DMOD}/TO_SOT_Packages_THT.3dshapes/TO-220-3_Horizontal.wrl
-      (at (xyz 0.1 0 0))
-      (scale (xyz 0.393701 0.393701 0.393701))
-      (rotate (xyz 0 0 0))
-    )
-  )
   (module Capacitors_SMD:C_0805 (layer B.Cu)
     (at 109.5 85)
@@
   (segment (start 96.981 117.994) (end 98.5 117.994) (width 0.25) (layer F.Cu) (net 435))
   (via (at 98.5 117.994) (size 0.3556) (drill 0.254) (layers F.Cu B.Cu) (net 435))
-  (segment (start 159 130.5) (end 160.5 129) (width 0.127) (layer B.Cu) (net 436))
+  (segment (start 160.5 130.5) (end 162 129) (width 0.127) (layer B.Cu) (net 436))
+  (segment (start 159 130.5) (end 160.5 130.5) (width 0.127) (layer B.Cu) (net 436))
   (segment (start 130 130.5) (end 159 130.5) (width 0.127) (layer B.Cu) (net 436))
   (segment (start 118.5 130.5) (end 130 130.5) (width 0.127) (layer B.Cu) (net 436))
@@
   (segment (start 102.066 123.074) (end 98.5 123.074) (width 0.25) (layer F.Cu) (net 436))
   (via (at 98.5 123.074) (size 0.3556) (drill 0.254) (layers F.Cu B.Cu) (net 436))
-  (segment (start 207 131) (end 209 129) (width 0.127) (layer B.Cu) (net 437))
-  (segment (start 205 131) (end 207 131) (width 0.127) (layer B.Cu) (net 437))
-  (segment (start 120 131) (end 205 131) (width 0.127) (layer B.Cu) (net 437))
-  (segment (start 116 131) (end 120 131) (width 0.127) (layer B.Cu) (net 437))
-  (segment (start 111.249 126.249) (end 116 131) (width 0.127) (layer B.Cu) (net 437))
+  (segment (start 206.4 131) (end 207.3 130.1) (width 0.127) (layer B.Cu) (net 437))
+  (segment (start 206 131) (end 206.4 131) (width 0.127) (layer B.Cu) (net 437))
+  (segment (start 205 131) (end 206 131) (width 0.127) (layer B.Cu) (net 437))
+  (via (at 98.5 126.249) (size 0.3556) (drill 0.254) (layers F.Cu B.Cu) (net 437))
   (segment (start 98.5 126.249) (end 111.249 126.249) (width 0.127) (layer B.Cu) (net 437))
+  (segment (start 111.249 126.249) (end 116 131) (width 0.127) (layer B.Cu) (net 437))
+  (segment (start 116 131) (end 120 131) (width 0.127) (layer B.Cu) (net 437))
+  (segment (start 120 131) (end 205 131) (width 0.127) (layer B.Cu) (net 437))
   (segment (start 98.5 126.249) (end 102.066 126.249) (width 0.25) (layer F.Cu) (net 437))
   (segment (start 96.981 126.249) (end 98.5 126.249) (width 0.25) (layer F.Cu) (net 437))
-  (via (at 98.5 126.249) (size 0.3556) (drill 0.254) (layers F.Cu B.Cu) (net 437))
   (segment (start 103 120.549) (end 96.996 120.549) (width 0.25) (layer F.Cu) (net 438))
   (segment (start 109.906 120.549) (end 103 120.549) (width 0.25) (layer F.Cu) (net 438))
@@
     (polygon
       (pts
-        (xy 68.5 111.5) (xy 88.5 111.5) (xy 88.5 129.5) (xy 68.5 129.5)
+        (xy 70 112) (xy 90 112) (xy 90 130) (xy 70 130)
       )
     )
@@
     (polygon
       (pts
-        (xy 123.5 111.584625) (xy 143.5 111.584625) (xy 143.5 129.584625) (xy 123.5 129.584625)
+        (xy 119 112) (xy 139 112) (xy 139 130) (xy 119 130)
       )
     )
@@
     (polygon
       (pts
-        (xy 160 111.5) (xy 180 111.5) (xy 180 129.5) (xy 160 129.5)
+        (xy 161 112) (xy 181 112) (xy 181 130) (xy 161 130)
       )
     )
@@
     (polygon
       (pts
-        (xy 208.5 111.5) (xy 228.5 111.5) (xy 228.5 129.5) (xy 208.5 129.5)
+        (xy 207 112.446511) (xy 227 112.446511) (xy 227 130.446511) (xy 207 130.446511)
       )
     )
